File: pcb/drumkid/drumkid.sch (KiCad schematic (older format))
At the start: 35 parts, among them J1 AudioJack3_Ground, SW1 SW_SPST, SW2 SW_SPST, SW3 SW_SPST, SW4 SW_SPST, SW5 SW_SPST, SW6 SW_SPST, SW7 SW_SPST, SW8 SW_SPST, U1 ATmega328P-PU, U2 MAX756, Y1 16MHz

Commit message: started PCB layout
Parts:
- removed J1: AudioJack3_Ground, symbol Connector:AudioJack3_Ground
- removed SW1: SW_SPST, symbol Switch:SW_SPST
- added J1: AudioJack3_Ground_Switch, headphone:Tayda_3.5mm_stereo_TRS_jack_A-853, symbol Connector:AudioJack3_Ground_Switch
- added SW1: SW_SPDT, Button_Switch_THT:SW_CuK_OS102011MA1QN1_SPDT_Angled, symbol Switch:SW_SPDT
- SW2, SW3, SW4, SW5, SW6, SW7, SW8: footprint (none) -> softtactile:SOFT_TACTILE_2
Connections:
- net GND: now also J1.S
- net at RV1.2: now also J1.R, J1.T
- net at BT1.1 (+): now also SW1.2 (B)
- net at C1.1, L1.1, U2.1 (~SHDN~)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: now also SW1.1 (A)
- no-connect marks 8 -> 11
Other:
- moved on the sheet: BT1
Changed lines of the file:
@@
-$EndComp
-$Comp
-L Connector:AudioJack3_Ground J1
-U 1 1 5C708CAA
-P 8600 3400
-F 0 "J1" H 8604 3742 50  0000 C CNN
-F 1 "AudioJack3_Ground" H 8604 3651 50  0000 C CNN
-F 2 "" H 8600 3400 50  0001 C CNN
-F 3 "~" H 8600 3400 50  0001 C CNN
-	1    8600 3400
-	-1   0    0    1
 $EndComp
 $Comp
@@
 F 0 "SW2" H 7550 5235 50  0000 C CNN
 F 1 "SW_SPST" H 7550 5144 50  0000 C CNN
-F 2 "" H 7550 5000 50  0001 C CNN
+F 2 "softtactile:SOFT_TACTILE_2" H 7550 5000 50  0001 C CNN
 F 3 "" H 7550 5000 50  0001 C CNN
 	1    7550 5000
@@
 F 0 "SW4" H 8000 5335 50  0000 C CNN
 F 1 "SW_SPST" H 8000 5244 50  0000 C CNN
-F 2 "" H 8000 5100 50  0001 C CNN
+F 2 "softtactile:SOFT_TACTILE_2" H 8000 5100 50  0001 C CNN
 F 3 "" H 8000 5100 50  0001 C CNN
 	1    8000 5100
@@
 F 0 "SW5" H 8450 5435 50  0000 C CNN
 F 1 "SW_SPST" H 8450 5344 50  0000 C CNN
-F 2 "" H 8450 5200 50  0001 C CNN
+F 2 "softtactile:SOFT_TACTILE_2" H 8450 5200 50  0001 C CNN
 F 3 "" H 8450 5200 50  0001 C CNN
 	1    8450 5200
@@
 F 0 "SW6" H 8900 5535 50  0000 C CNN
 F 1 "SW_SPST" H 8900 5444 50  0000 C CNN
-F 2 "" H 8900 5300 50  0001 C CNN
+F 2 "softtactile:SOFT_TACTILE_2" H 8900 5300 50  0001 C CNN
 F 3 "" H 8900 5300 50  0001 C CNN
 	1    8900 5300
@@
 F 0 "SW7" H 9350 5635 50  0000 C CNN
 F 1 "SW_SPST" H 9350 5544 50  0000 C CNN
-F 2 "" H 9350 5400 50  0001 C CNN
+F 2 "softtactile:SOFT_TACTILE_2" H 9350 5400 50  0001 C CNN
 F 3 "" H 9350 5400 50  0001 C CNN
 	1    9350 5400
@@
 F 0 "SW8" H 9800 5735 50  0000 C CNN
 F 1 "SW_SPST" H 9800 5644 50  0000 C CNN
-F 2 "" H 9800 5500 50  0001 C CNN
+F 2 "softtactile:SOFT_TACTILE_2" H 9800 5500 50  0001 C CNN
 F 3 "" H 9800 5500 50  0001 C CNN
 	1    9800 5500
@@
 F 0 "SW3" H 7850 3085 50  0000 C CNN
 F 1 "SW_SPST" H 7850 2994 50  0000 C CNN
-F 2 "" H 7850 2850 50  0001 C CNN
+F 2 "softtactile:SOFT_TACTILE_2" H 7850 2850 50  0001 C CNN
 F 3 "" H 7850 2850 50  0001 C CNN
 	1    7850 2850
@@
 Wire Wire Line
 	7450 3500 8100 3500
-Wire Wire Line
-	8100 3500 8400 3500
 Connection ~ 8100 3500
 Wire Wire Line
 	8250 3350 8400 3350
-Wire Wire Line
-	8400 3350 8400 3300
 Wire Wire Line
 	8400 3400 8400 3350
@@
 L Device:Battery BT1
 U 1 1 5C8C17C6
-P 1000 1950
-F 0 "BT1" H 1108 1996 50  0000 L CNN
-F 1 "Battery" H 1108 1905 50  0000 L CNN
-F 2 "Connector_PinHeader_2.54mm:PinHeader_1x02_P2.54mm_Vertical" V 1000 2010 50  0001 C CNN
-F 3 "~" V 1000 2010 50  0001 C CNN
-	1    1000 1950
+P 750 1950
+F 0 "BT1" H 858 1996 50  0000 L CNN
+F 1 "Battery" H 858 1905 50  0000 L CNN
+F 2 "Connector_PinHeader_2.54mm:PinHeader_1x02_P2.54mm_Vertical" V 750 2010 50  0001 C CNN
+F 3 "~" V 750 2010 50  0001 C CNN
+	1    750  1950
 	1    0    0    -1
 $EndComp
@@
 	1400 2300 1700 2300
 Connection ~ 1700 2300
-$Comp
-L Switch:SW_SPST SW1
-U 1 1 5C8C4B20
-P 1200 1500
-F 0 "SW1" H 1200 1735 50  0000 C CNN
-F 1 "SW_SPST" H 1200 1644 50  0000 C CNN
-F 2 "" H 1200 1500 50  0001 C CNN
-F 3 "" H 1200 1500 50  0001 C CNN
-	1    1200 1500
-	1    0    0    -1
-$EndComp
-Wire Wire Line
-	1000 2300 1000 2150
-Wire Wire Line
-	1000 1750 1000 1500
-Wire Wire Line
-	1400 1500 1400 1600
+Wire Wire Line
+	750  2300 750  2150
+Wire Wire Line
+	750  1750 750  1500
 $Comp
 L pspice:INDUCTOR L1
@@
 Wire Wire Line
 	3000 1000 2500 1000
-Wire Wire Line
-	1400 1000 1400 1500
-Connection ~ 1400 1500
 $Comp
 L Diode:1N5817 D1
@@
 	1    0    0    -1
 $EndComp
-Connection ~ 1400 2300
-Wire Wire Line
-	1400 2300 1000 2300
 $Comp
 L power:PWR_FLAG #FLG0101
@@
 NoConn ~ 4450 4400
 NoConn ~ 4450 4500
+$Comp
+L Switch:SW_SPDT SW1
+U 1 1 5C93A215
+P 950 1500
+F 0 "SW1" H 950 1785 50  0000 C CNN
+F 1 "SW_SPDT" H 950 1694 50  0000 C CNN
+F 2 "Button_Switch_THT:SW_CuK_OS102011MA1QN1_SPDT_Angled" H 950 1500 50  0001 C CNN
+F 3 "" H 950 1500 50  0001 C CNN
+	1    950  1500
+	1    0    0    -1
+$EndComp
+Wire Wire Line
+	1400 1000 1400 1400
+Wire Wire Line
+	750  2300 1400 2300
+Connection ~ 1400 2300
+Wire Wire Line
+	1150 1400 1400 1400
+Connection ~ 1400 1400
+Wire Wire Line
+	1400 1400 1400 1600
+NoConn ~ 1150 1600
+$Comp
+L Connector:AudioJack3_Ground_Switch J1
+U 1 1 5C93B028
+P 8750 3400
+F 0 "J1" H 8517 3279 50  0000 R CNN
+F 1 "AudioJack3_Ground_Switch" H 8517 3370 50  0000 R CNN
+F 2 "headphone:Tayda_3.5mm_stereo_TRS_jack_A-853" H 8750 3400 50  0001 C CNN
+F 3 "~" H 8750 3400 50  0001 C CNN
+	1    8750 3400
+	-1   0    0    1
+$EndComp
+Wire Wire Line
+	8100 3500 8550 3500
+Wire Wire Line
+	8400 3400 8550 3400
+Wire Wire Line
+	8400 3200 8550 3200
+Wire Wire Line
+	8400 3200 8400 3350
+NoConn ~ 8550 3300
+NoConn ~ 8550 3100
 $EndSCHEMATC
