File: pcb/drumkid/drumkid.kicad_pcb (KiCad board)
At the start: 2 copper layers, 35 parts, among them J1 AudioJack3_Ground_Switch, SW1 SW_SPDT, SW2 SW_SPST, SW3 SW_SPST, SW4 SW_SPST, SW5 SW_SPST, SW6 SW_SPST, SW7 SW_SPST, SW8 SW_SPST, U1 ATmega328P-PU, U2 MAX756, Y1 16MHz

Commit message: pcb layout looking nice-ish
Parts:
- moved R6 143.0 mm to (47.5, 72.5)
- moved D1 125.0 mm to (115.0, 42.5)
- moved L1 114.9 mm to (122.5, 35.0)
- moved C6 113.7 mm to (122.5, 52.5)
- moved C1 111.3 mm to (112.5, 52.5)
- moved U2 102.5 mm to (97.5, 47.5)
- moved C2 98.2 mm to (90.0, 52.5), turned to 90 degrees
- moved R4 97.0 mm to (61.5, 72.5)
- moved R3 78.3 mm to (90.0, 57.5), turned to 180 degrees
- moved R5 74.9 mm to (122.5, 72.5), turned to 180 degrees
- moved SW8 74.3 mm to (120.0, 100.0)
- moved SW5 71.5 mm to (120.0, 85.0)
- moved SW2 65.2 mm to (107.5, 90.0)
- moved SW6 64.7 mm to (107.5, 105.0)
- moved R7 56.2 mm to (107.5, 72.5), turned to 180 degrees
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Other:
- board outline added: 85 x 95 mm

Commit message: quick commit before i finalise the layout
Parts:
- moved R4 11.4 mm to (72.9, 72.5), turned to 180 degrees
- moved R5 10.7 mm to (111.8, 72.5), turned to 0 degrees
- moved R7 9.96 mm to (97.5, 72.5), turned to 0 degrees
- moved R6 9.90 mm to (57.4, 72.5), turned to 180 degrees
Routing:
- net +5V: track 0.00 -> 155.0 mm
- net Net-(R1-Pad2): track 0.00 -> 123.9 mm
- net Net-(BT1-Pad1): track 0.00 -> 111.7 mm
- net Net-(R6-Pad2): track 0.00 -> 107.7 mm
- net Net-(R4-Pad2): track 0.00 -> 106.6 mm
- net Net-(R5-Pad2): track 0.00 -> 77.2 mm
- net Net-(SW4-Pad1): track 0.00 -> 76.2 mm
- net Net-(J1-PadR): track 0.00 -> 56.6 mm
- net Net-(C1-Pad1): track 0.00 -> 55.0 mm
- net Net-(R7-Pad2): track 0.00 -> 47.1 mm
- net Net-(C3-Pad2): track 0.00 -> 46.8 mm
- net Net-(RV2-Pad2): track 0.00 -> 45.3 mm
- net Net-(SW8-Pad1): track 0.00 -> 44.6 mm
- net Net-(R3-Pad2): track 0.00 -> 44.4 mm
- net Net-(SW5-Pad1): track 0.00 -> 41.7 mm
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