File: pcb/drumkid/drumkid.kicad_pcb (KiCad board)
At the start: 2 copper layers, 85 x 95 mm, 35 parts, among them J1 AudioJack3_Ground_Switch, SW1 SW_SPDT, SW2 SW_SPST, SW3 SW_SPST, SW4 SW_SPST, SW5 SW_SPST, SW6 SW_SPST, SW7 SW_SPST, SW8 SW_SPST, U1 ATmega328P-PU, U2 MAX756, Y1 16MHz

Commit message: layout finalised, gerbers generated, boards in production!
Other:
- board text added: "DrumKid v01 by Matt Bradshaw mattbradshawdesign.com"
Changed lines of the file:
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@@
   (general
     (thickness 1.6)
-    (drawings 21)
+    (drawings 22)
     (tracks 183)
     (zones 0)
@@
   )
   (layers
-    (0 F.Cu signal hide)
+    (0 F.Cu signal)
     (31 B.Cu signal)
     (32 B.Adhes user)
@@
     (visible_elements FFFFFF7F)
     (pcbplotparams
-      (layerselection 0x010fc_ffffffff)
+      (layerselection 0x010f0_ffffffff)
       (usegerberextensions false)
       (usegerberattributes false)
@@
       (outputformat 1)
       (mirror false)
-      (drillshape 1)
+      (drillshape 0)
       (scaleselection 1)
-      (outputdirectory ""))
+      (outputdirectory "gerbers/"))
   )
   (net 0 "")
@@
     (add_net "Net-(U1-Pad3)")
     (add_net "Net-(U2-Pad4)")
+  )
+  (module headphone:Tayda_3.5mm_stereo_TRS_jack_A-853 (layer F.Cu)
+    (at 67.5 36.424)
+    (fp_text reference J1 (at -4.318 7.112) (layer F.SilkS)
+      (effects (font (size 0.8 0.8) (thickness 0.15)))
+    )
+    (fp_text value AudioJack3_Ground_Switch (at 0 0.508) (layer F.SilkS)
+      (effects (font (size 0.6 0.6) (thickness 0.1)))
+    )
+    (fp_line (start -1.778 -1.524) (end -3.81 -1.524) (layer F.SilkS) (width 0.15))
+    (fp_line (start -3.81 -1.524) (end -3.81 -5.08) (layer F.SilkS) (width 0.15))
+    (fp_line (start -3.81 -5.08) (end 3.81 -5.08) (layer F.SilkS) (width 0.15))
+    (fp_line (start 3.81 -5.08) (end 3.81 -1.524) (layer F.SilkS) (width 0.15))
+    (fp_line (start 3.81 -1.524) (end 1.778 -1.524) (layer F.SilkS) (width 0.15))
+    (fp_line (start -5.08 -6.096) (end -6.096 -6.096) (layer F.SilkS) (width 0.15))
+    (fp_line (start 6.096 -6.096) (end 5.08 -6.096) (layer F.SilkS) (width 0.15))
+    (fp_line (start -2.54 -8.128) (end -2.54 -6.604) (layer F.SilkS) (width 0.15))
+    (fp_line (start 2.54 -6.604) (end 2.54 -8.128) (layer F.SilkS) (width 0.15))
+    (fp_line (start -2.54 -7.366) (end 2.54 -7.366) (layer F.SilkS) (width 0.15))
+    (fp_line (start -5.08 -6.096) (end -5.08 -6.35) (layer F.SilkS) (width 0.15))
+    (fp_line (start -5.08 -6.35) (end -5.08 -6.604) (layer F.SilkS) (width 0.15))
+    (fp_line (start -5.08 -6.604) (end 5.08 -6.604) (layer F.SilkS) (width 0.15))
+    (fp_line (start 5.08 -6.604) (end 5.08 -6.096) (layer F.SilkS) (width 0.15))
+    (fp_line (start -2.54 -8.128) (end 2.54 -8.128) (layer F.SilkS) (width 0.15))
+    (fp_line (start -6.096 6.096) (end -6.096 -6.096) (layer F.SilkS) (width 0.15))
+    (fp_line (start 6.096 -6.096) (end 6.096 6.096) (layer F.SilkS) (width 0.15))
+    (fp_line (start 6.096 6.096) (end -6.096 6.096) (layer F.SilkS) (width 0.15))
+    (pad S thru_hole rect (at 0 -1.596) (size 3.5 2.5) (drill 1.2) (layers *.Cu *.Mask F.SilkS)
+      (net 2 GND))
+    (pad R thru_hole oval (at 5 3.41) (size 1.75 3.5) (drill 1.2) (layers *.Cu *.Mask F.SilkS)
+      (net 15 "Net-(J1-PadR)"))
+    (pad T thru_hole oval (at -5 3.41) (size 1.75 3.5) (drill 1.2) (layers *.Cu *.Mask F.SilkS)
+      (net 15 "Net-(J1-PadR)"))
+    (pad RN thru_hole oval (at 2.5 3.41) (size 1.75 3.5) (drill 1.2) (layers *.Cu *.Mask F.SilkS)
+      (net 16 "Net-(J1-PadRN)"))
+    (pad TN thru_hole oval (at -2.5 3.41) (size 1.75 3.5) (drill 1.2) (layers *.Cu *.Mask F.SilkS)
+      (net 17 "Net-(J1-PadTN)"))
   )
   (module Connector_PinHeader_2.54mm:PinHeader_1x02_P2.54mm_Vertical (layer F.Cu)
@@
     )
   )
-  (module headphone:Tayda_3.5mm_stereo_TRS_jack_A-853 (layer F.Cu)
-    (at 67.5 36.424)
-    (fp_text reference J1 (at -4.318 7.112) (layer F.SilkS)
-      (effects (font (size 0.8 0.8) (thickness 0.15)))
-    )
-    (fp_text value AudioJack3_Ground_Switch (at 0 0.508) (layer F.SilkS)
-      (effects (font (size 0.6 0.6) (thickness 0.1)))
-    )
-    (fp_line (start -1.778 -1.524) (end -3.81 -1.524) (layer F.SilkS) (width 0.15))
-    (fp_line (start -3.81 -1.524) (end -3.81 -5.08) (layer F.SilkS) (width 0.15))
-    (fp_line (start -3.81 -5.08) (end 3.81 -5.08) (layer F.SilkS) (width 0.15))
-    (fp_line (start 3.81 -5.08) (end 3.81 -1.524) (layer F.SilkS) (width 0.15))
-    (fp_line (start 3.81 -1.524) (end 1.778 -1.524) (layer F.SilkS) (width 0.15))
-    (fp_line (start -5.08 -6.096) (end -6.096 -6.096) (layer F.SilkS) (width 0.15))
-    (fp_line (start 6.096 -6.096) (end 5.08 -6.096) (layer F.SilkS) (width 0.15))
-    (fp_line (start -2.54 -8.128) (end -2.54 -6.604) (layer F.SilkS) (width 0.15))
-    (fp_line (start 2.54 -6.604) (end 2.54 -8.128) (layer F.SilkS) (width 0.15))
-    (fp_line (start -2.54 -7.366) (end 2.54 -7.366) (layer F.SilkS) (width 0.15))
-    (fp_line (start -5.08 -6.096) (end -5.08 -6.35) (layer F.SilkS) (width 0.15))
-    (fp_line (start -5.08 -6.35) (end -5.08 -6.604) (layer F.SilkS) (width 0.15))
-    (fp_line (start -5.08 -6.604) (end 5.08 -6.604) (layer F.SilkS) (width 0.15))
-    (fp_line (start 5.08 -6.604) (end 5.08 -6.096) (layer F.SilkS) (width 0.15))
-    (fp_line (start -2.54 -8.128) (end 2.54 -8.128) (layer F.SilkS) (width 0.15))
-    (fp_line (start -6.096 6.096) (end -6.096 -6.096) (layer F.SilkS) (width 0.15))
-    (fp_line (start 6.096 -6.096) (end 6.096 6.096) (layer F.SilkS) (width 0.15))
-    (fp_line (start 6.096 6.096) (end -6.096 6.096) (layer F.SilkS) (width 0.15))
-    (pad S thru_hole rect (at 0 -1.596) (size 3.5 2.5) (drill 1.2) (layers *.Cu *.Mask F.SilkS)
-      (net 2 GND))
-    (pad R thru_hole oval (at 5 3.41) (size 1.75 3.5) (drill 1.2) (layers *.Cu *.Mask F.SilkS)
-      (net 15 "Net-(J1-PadR)"))
-    (pad T thru_hole oval (at -5 3.41) (size 1.75 3.5) (drill 1.2) (layers *.Cu *.Mask F.SilkS)
-      (net 15 "Net-(J1-PadR)"))
-    (pad RN thru_hole oval (at 2.5 3.41) (size 1.75 3.5) (drill 1.2) (layers *.Cu *.Mask F.SilkS)
-      (net 16 "Net-(J1-PadRN)"))
-    (pad TN thru_hole oval (at -2.5 3.41) (size 1.75 3.5) (drill 1.2) (layers *.Cu *.Mask F.SilkS)
-      (net 17 "Net-(J1-PadTN)"))
-  )
   (module Inductor_THT:L_Radial_D6.0mm_P4.00mm (layer F.Cu)
     (at 122.5 35)
@@
     )
   )
+  (gr_text "DrumKid v01\nby Matt Bradshaw\nmattbradshawdesign.com" (at 90 37.5) (layer F.SilkS)
+    (effects (font (size 1.5 1.5) (thickness 0.3)))
+  )
   (gr_circle (center 86.5 78.5) (end 91.5 78.5) (layer Dwgs.User) (width 0.2))
