File: pcb/drumkid v2/drumkid v2.sch (KiCad schematic (older format))
At the start: 43 parts, among them J1 Conn_01x03_Female, J2 Conn_01x03_Female, J3 Conn_01x03_Female, J4 Conn_01x03_Female, J5 Conn_01x05_Female, J6 Conn_01x04_Female, J7 Conn_01x06_Female, J8 Conn_01x05_Female, J9 AudioJack3_Ground_Switch, SW1 SW_SPDT, SW2 SW_Push, SW3 SW_Push, SW4 SW_Push, SW5 SW_Push, SW6 SW_Push, U1 MAX756, U2 ATmega328P-PU, Y1 Crystal

Commit message: more pcb changes, about to do a big-ish change so doing a commit now
Parts:
- added C10: 220uF, Capacitor_THT:CP_Radial_D6.3mm_P2.50mm, symbol Device:CP
- added C7: 10uF, Capacitor_THT:CP_Radial_D6.3mm_P2.50mm, symbol Device:CP
- added C8: 100uF, Capacitor_THT:CP_Radial_D6.3mm_P2.50mm, symbol Device:CP
- added C9: 0.1uF, Capacitor_THT:C_Disc_D3.4mm_W2.1mm_P2.50mm, symbol Device:C
- added R10: 100k, Resistor_THT:R_Axial_DIN0207_L6.3mm_D2.5mm_P10.16mm_Horizontal, symbol Device:R
- added R8: 10, Resistor_THT:R_Axial_DIN0207_L6.3mm_D2.5mm_P10.16mm_Horizontal, symbol Device:R
- added R9: 470k, Resistor_THT:R_Axial_DIN0207_L6.3mm_D2.5mm_P10.16mm_Horizontal, symbol Device:R
- added U3: LM386, Package_DIP:DIP-8_W7.62mm_Socket, symbol Amplifier_Audio:LM386
- C1: value CP -> 150uF
- C2, C4: value C -> 0.1uF
- C3: value CP -> 100uF
- C5, C6: value C -> 10uF
- R1: value R -> 470
- R2: value R -> 10k
- R3, R4, R5, R6, R7: value R -> 220
- U1: footprint MAX756:SO08 -> Package_DIP:DIP-8_W7.62mm_Socket
- U2: footprint Package_DIP:DIP-28_W7.62mm -> Package_DIP:DIP-28_W7.62mm_Socket
Connections:
- net +5V: now also C8.1, U3.6 (V+)
- net GND: now also C5.2, C6.2, RV1.1, C7.2, C8.2, R10.1, R8.1, U3.2 (-), U3.4 (GND); no longer RV1.3
- net at C4.2, R1.2: now also R9.1; no longer RV1.1
- net at J9.R, J9.T: now also C10.2; no longer RV1.2
- new net: RV1.2, U3.3 (+)
- new net: R10.2, R9.2, RV1.3
- new net: C10.1, C9.1, U3.5
- new net: C7.1, U3.7 (BYPASS)
- new net: C9.2, R8.2
- no-connect marks 5 -> 7
Other:
- moved on the sheet: BT1, C1, C2, C3, C4, C5, C6, D1, D2, D3, D4, D5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

Commit message: good pcb progress, about to make a little change
Parts:
- removed J1, J2, J3, J4: Conn_01x03_Female, Connector_PinHeader_2.54mm:PinHeader_1x03_P2.54mm_Vertical, symbol Connector:Conn_01x03_Female
- added C11, C12: CP, Capacitor_THT:CP_Radial_D6.3mm_P2.50mm, symbol Device:CP
- added C13: 2.2uF, Capacitor_THT:CP_Radial_D6.3mm_P2.50mm, symbol Device:CP
- added C14: 220nF, Capacitor_THT:C_Disc_D3.4mm_W2.1mm_P2.50mm, symbol Device:C
- added C15, C17: 10uF, Capacitor_THT:CP_Radial_D6.3mm_P2.50mm, symbol Device:CP
- added C16, C18: 100nF, Capacitor_THT:C_Disc_D3.4mm_W2.1mm_P2.50mm, symbol Device:C
- added R11: 10, Resistor_THT:R_Axial_DIN0207_L6.3mm_D2.5mm_P10.16mm_Horizontal, symbol Device:R
- C4, C9: value 0.1uF -> C
- C7: value 10uF -> CP
- C8: value 100uF -> CP
- R1: value 470 -> 47
- R10: value 100k -> 1k
- R8: value 10 -> 470
- R9: value 470k -> 10k
- RV1: value R_POT -> 10k; footprint SamacSys_Parts:RK14J12A0A0K -> Resistor_THT:R_Axial_DIN0207_L6.3mm_D2.5mm_P10.16mm_Horizontal
Connections:
- net +5V: now also C4.2, C7.1, C9.2, C11.1, C12.1, C16.1
- net DIGITAL_9: now also R1.2; no longer R1.1
- net GND: now also C9.1, R10.2, C11.2, C12.2, C13.2, C14.2, C17.1, R11.2; no longer R10.1, R8.1, RV1.1, U3.2 (-), U3.4 (GND)
- net at C10.1, U3.5: now also C18.1; no longer C9.1
- net at U3.7 (BYPASS): now also C17.2; no longer C7.1
- net at R8.2: now also R1.1, C13.1; no longer C9.2
- new net: R10.1, R9.1, RV1.3
- new net: C15.2, R9.2
- new net: C14.1, C15.1, R8.1
- new net: C18.2, R11.1
- new net: C16.2, U3.4 (GND)
- new net: RV1.1, U3.2 (-)
Other:
- note added: "Arduino pin breakouts for extra hackability"
- note added: "Atmega328 decoupling capacitors"
- note added: "Voltage boost from 3V to 5V"
- moved on the sheet: BT1, C1, C10, C2, C3, D1, J9, L1, SW1, U1

Commit message: layout done? ready to route tracks
Parts:
- added J1: Conn_01x04_Female, Connector_PinHeader_2.54mm:PinHeader_1x04_P2.54mm_Vertical, symbol Connector:Conn_01x04_Female
- added SW7: SW_Push, Button_Switch_THT:SW_PUSH-12mm_Wuerth-430476085716, symbol Switch:SW_Push
- RV1: footprint Resistor_THT:R_Axial_DIN0207_L6.3mm_D2.5mm_P10.16mm_Horizontal -> SamacSys_Parts:RK14J12A0A0K
Connections:
- net +5V: now also J1.1 (Pin_1), J1.2 (Pin_2)
- net DIGITAL_13: now also SW7.1
- net GND: now also RV1.1, U3.2 (-), J1.3 (Pin_3), J1.4 (Pin_4), SW7.2
- net at R10.1, R9.1: now also U3.3 (+); no longer RV1.3
- net at R9.2: now also RV1.2; no longer C15.2
- new net: C15.2, RV1.3
Other:
- moved on the sheet: C5, C6, D2, D3, D4, D5, D6, R10, R3, R4, R5, R6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

Commit message: routing half done maybe
Connections:
- net GND: now also C17.2; no longer C17.1
- net BAT_ON: now reaches C1.1, L1.1, SW1.1 (A), U1.1 (~SHDN~), U1.5 (LBI)
- net at U3.7 (BYPASS): now also C17.1; no longer C17.2
Other:
- moved on the sheet: C17
Changed lines of the file:
@@
 L Device:CP C17
 U 1 1 5CD6A157
-P 8050 850
-F 0 "C17" V 7795 850 50  0000 C CNN
-F 1 "10uF" V 7886 850 50  0000 C CNN
-F 2 "Capacitor_THT:CP_Radial_D6.3mm_P2.50mm" H 8088 700 50  0001 C CNN
-F 3 "~" H 8050 850 50  0001 C CNN
-	1    8050 850
-	0    1    1    0
+P 8200 850
+F 0 "C17" V 8455 850 50  0000 C CNN
+F 1 "10uF" V 8364 850 50  0000 C CNN
+F 2 "Capacitor_THT:CP_Radial_D6.3mm_P2.50mm" H 8238 700 50  0001 C CNN
+F 3 "~" H 8200 850 50  0001 C CNN
+	1    8200 850
+	0    -1   -1   0
 $EndComp
 $Comp
@@
 	9050 1150 9100 1150
 Wire Wire Line
-	8200 850  8600 850
-Wire Wire Line
 	8600 850  8600 1900
 Wire Wire Line
@@
 Wire Wire Line
 	7300 3700 7300 4200
+Text Label 1350 900  1    50   ~ 0
+BAT_ON
+Wire Wire Line
+	8350 850  8600 850
+Wire Wire Line
+	7900 850  8050 850
 $EndSCHEMATC

Commit message: everything working pretty nicely
Parts:
- C5, C6: value 10uF -> 22pF
Changed lines of the file:
@@
 P 8050 4200
 F 0 "C6" V 8302 4200 50  0000 C CNN
-F 1 "10uF" V 8211 4200 50  0000 C CNN
+F 1 "22pF" V 8211 4200 50  0000 C CNN
 F 2 "Capacitor_THT:C_Disc_D3.4mm_W2.1mm_P2.50mm" H 8088 4050 50  0001 C CNN
 F 3 "~" H 8050 4200 50  0001 C CNN
@@
 P 8050 3800
 F 0 "C5" V 8302 3800 50  0000 C CNN
-F 1 "10uF" V 8211 3800 50  0000 C CNN
+F 1 "22pF" V 8211 3800 50  0000 C CNN
 F 2 "Capacitor_THT:C_Disc_D3.4mm_W2.1mm_P2.50mm" H 8088 3650 50  0001 C CNN
 F 3 "~" H 8050 3800 50  0001 C CNN
