File: pcb/drumkid v4/drumkid v3.kicad_pcb (KiCad board)
At the start: 2 copper layers, 90 x 120 mm, 61 parts, among them J1 Conn_01x04_Female, J5 Conn_01x05_Female, J6 Conn_01x04_Female, J7 Conn_01x06_Female, J8 Conn_01x05_Female, J9 AudioJack3_Ground_Switch, SW1 SW_SPDT, SW2 SW_Push, SW3 SW_Push, SW4 SW_Push, SW5 SW_Push, SW6 SW_Push, SW7 SW_Push, U2 ATmega328P-PU, U3 LM386, Y1 Crystal

Commit message: v4 progress...
Parts:
- moved C13 113.1 mm to (142.2, 152.4)
- moved C15 111.4 mm to (134.6, 152.4)
- moved C16 69.1 mm to (137.2, 147.3)
- moved C18 67.5 mm to (132.0, 147.3)
- moved C17 63.0 mm to (114.3, 132.1)
- moved C10 48.7 mm to (119.4, 124.5)
- moved BT1 33.6 mm to (119.4, 116.8)
- moved C5 10.2 mm to (149.9, 116.8)
- moved J8 10.2 mm to (149.9, 142.2)
- moved Y1 10.2 mm to (149.9, 121.9)
- moved R10 10.2 mm to (134.6, 142.2)
- moved R11 10.2 mm to (134.6, 139.7)
- moved C12 10.2 mm to (160.0, 119.4)
- moved C4 10.2 mm to (165.1, 129.5)
- moved C6 10.2 mm to (142.2, 116.8)
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
Commit message: v4 looking good, about to start routing
Parts:
- BT1: footprint Connector_PinHeader_2.54mm:PinHeader_1x02_P2.54mm_Vertical -> Connector_Wire:SolderWirePad_1x02_P5.08mm_Drill1.5mm
- moved BT1 2.54 mm to (116.8, 116.8), turned to 0 degrees
Routing:
- removed copper zone on B.Cu, net GND
- removed copper zone on F.Cu, net GND
Other:
- board text added: "A"
- board text added: "B"
- board text added: "C"
- board text added: "X"
- board text added: "Y"
- board text added: "Z"
Changed lines of the file:
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@@
   (general
     (thickness 1.6)
-    (drawings 19)
+    (drawings 25)
     (tracks 0)
     (zones 0)
@@
     (add_net "Net-(BT1-Pad1)")
   )
+  (module Connector_Wire:SolderWirePad_1x02_P5.08mm_Drill1.5mm (layer F.Cu)
+    (at 116.84 116.84)
+    (descr "Wire solder connection")
+    (tags connector)
+    (attr virtual)
+    (fp_text reference BT1 (at 2.54 -3.81) (layer F.SilkS)
+      (effects (font (size 1 1) (thickness 0.15)))
+    )
+    (fp_text value Battery (at 2.54 3.81) (layer F.Fab)
+      (effects (font (size 1 1) (thickness 0.15)))
+    )
+    (fp_line (start 7.33 2.25) (end -2.25 2.25) (layer F.CrtYd) (width 0.05))
+    (fp_line (start 7.33 2.25) (end 7.33 -2.25) (layer F.CrtYd) (width 0.05))
+    (fp_line (start -2.25 -2.25) (end -2.25 2.25) (layer F.CrtYd) (width 0.05))
+    (fp_line (start -2.25 -2.25) (end 7.33 -2.25) (layer F.CrtYd) (width 0.05))
+    (fp_text user %R (at 2.54 0) (layer F.Fab)
+      (effects (font (size 1 1) (thickness 0.15)))
+    )
+    (pad 2 thru_hole circle (at 5.08 0) (size 3.50012 3.50012) (drill 1.50114) (layers *.Cu *.Mask)
+      (net 1 GND))
+    (pad 1 thru_hole rect (at 0 0) (size 3.50012 3.50012) (drill 1.50114) (layers *.Cu *.Mask)
+      (net 6 "Net-(BT1-Pad1)"))
+  )
   (module headphone:EG1206_NOSILK (layer B.Cu)
     (at 113.993946 60.991091 90)
@@
     (pad 1 np_thru_hole circle (at 0 0) (size 3.2 3.2) (drill 3.2) (layers *.Cu *.Mask))
   )
-  (module Connector_PinHeader_2.54mm:PinHeader_1x02_P2.54mm_Vertical (layer F.Cu)
-    (at 119.38 116.84 90)
-    (descr "Through hole straight pin header, 1x02, 2.54mm pitch, single row")
-    (tags "Through hole pin header THT 1x02 2.54mm single row")
-    (fp_text reference BT1 (at 0 -2.33 90) (layer F.SilkS)
-      (effects (font (size 1 1) (thickness 0.15)))
-    )
-    (fp_text value Battery (at 0 4.87 90) (layer F.Fab)
-      (effects (font (size 1 1) (thickness 0.15)))
-    )
-    (fp_line (start -0.635 -1.27) (end 1.27 -1.27) (layer F.Fab) (width 0.1))
-    (fp_line (start 1.27 -1.27) (end 1.27 3.81) (layer F.Fab) (width 0.1))
-    (fp_line (start 1.27 3.81) (end -1.27 3.81) (layer F.Fab) (width 0.1))
-    (fp_line (start -1.27 3.81) (end -1.27 -0.635) (layer F.Fab) (width 0.1))
-    (fp_line (start -1.27 -0.635) (end -0.635 -1.27) (layer F.Fab) (width 0.1))
-    (fp_line (start -1.33 3.87) (end 1.33 3.87) (layer F.SilkS) (width 0.12))
-    (fp_line (start -1.33 1.27) (end -1.33 3.87) (layer F.SilkS) (width 0.12))
-    (fp_line (start 1.33 1.27) (end 1.33 3.87) (layer F.SilkS) (width 0.12))
-    (fp_line (start -1.33 1.27) (end 1.33 1.27) (layer F.SilkS) (width 0.12))
-    (fp_line (start -1.33 0) (end -1.33 -1.33) (layer F.SilkS) (width 0.12))
-    (fp_line (start -1.33 -1.33) (end 0 -1.33) (layer F.SilkS) (width 0.12))
-    (fp_line (start -1.8 -1.8) (end -1.8 4.35) (layer F.CrtYd) (width 0.05))
-    (fp_line (start -1.8 4.35) (end 1.8 4.35) (layer F.CrtYd) (width 0.05))
-    (fp_line (start 1.8 4.35) (end 1.8 -1.8) (layer F.CrtYd) (width 0.05))
-    (fp_line (start 1.8 -1.8) (end -1.8 -1.8) (layer F.CrtYd) (width 0.05))
-    (fp_text user %R (at 0 1.27 180) (layer F.Fab)
-      (effects (font (size 1 1) (thickness 0.15)))
-    )
-    (pad 1 thru_hole rect (at 0 0 90) (size 1.7 1.7) (drill 1) (layers *.Cu *.Mask)
-      (net 6 "Net-(BT1-Pad1)"))
-    (pad 2 thru_hole oval (at 0 2.54 90) (size 1.7 1.7) (drill 1) (layers *.Cu *.Mask)
-      (net 1 GND))
-    (model ${KISYS3DMOD}/Connector_PinHeader_2.54mm.3dshapes/PinHeader_1x02_P2.54mm_Vertical.wrl
-      (at (xyz 0 0 0))
-      (scale (xyz 1 1 1))
-      (rotate (xyz 0 0 0))
-    )
-  )
   (module Capacitor_THT:CP_Radial_D6.3mm_P2.50mm (layer F.Cu)
     (at 149.86 152.4)
@@
     (pad 1 np_thru_hole circle (at 0 0) (size 3.2 3.2) (drill 3.2) (layers *.Cu *.Mask))
   )
+  (gr_text Z (at 112.522 104.648) (layer B.SilkS)
+    (effects (font (size 1.5 1.5) (thickness 0.3)) (justify mirror))
+  )
+  (gr_text Y (at 125.73 104.648) (layer B.SilkS)
+    (effects (font (size 1.5 1.5) (thickness 0.3)) (justify mirror))
+  )
+  (gr_text X (at 138.684 104.648) (layer B.SilkS)
+    (effects (font (size 1.5 1.5) (thickness 0.3)) (justify mirror))
+  )
+  (gr_text C (at 161.544 104.648) (layer B.SilkS)
+    (effects (font (size 1.5 1.5) (thickness 0.3)) (justify mirror))
+  )
+  (gr_text B (at 174.752 104.648) (layer B.SilkS)
+    (effects (font (size 1.5 1.5) (thickness 0.3)) (justify mirror))
+  )
+  (gr_text A (at 187.706 104.648) (layer B.SilkS)
+    (effects (font (size 1.5 1.5) (thickness 0.3)) (justify mirror))
+  )
   (gr_line (start 121 114) (end 121 66) (layer Dwgs.User) (width 0.2))
   (gr_line (start 179 114) (end 121 114) (layer Dwgs.User) (width 0.2))
@@
     (effects (font (size 1.5 1.5) (thickness 0.3)))
   )
-  (gr_line (start 150 42.54) (end 150 162.54) (layer Dwgs.User) (width 0.2))
+  (gr_line (start 150 40) (end 150 160) (layer Dwgs.User) (width 0.2))
   (gr_text drumkid (at 149.86 57.15) (layer B.SilkS)
     (effects (font (size 7 7) (thickness 1.5)) (justify mirror))
   )
-  (gr_text "B+\nB-" (at 88.07 130.32 90) (layer F.SilkS)
+  (gr_text "B+\n\nB-" (at 119.38 114.3 90) (layer F.SilkS)
     (effects (font (size 1.5 1.5) (thickness 0.3)) (justify left))
   )
@@
   (gr_line (start 109.993946 39.991091) (end 189.993946 39.991091) (layer Edge.Cuts) (width 0.1))
   (gr_line (start 104.993946 44.991091) (end 104.993946 129.991091) (layer Edge.Cuts) (width 0.1))
-  (zone (net 1) (net_name GND) (layer B.Cu) (hatch edge 0.508)
-    (connect_pads (clearance 0.508))
-    (min_thickness 0.254)
-    (fill (arc_segments 16) (thermal_gap 0.508) (thermal_bridge_width 0.508))
-    (polygon
-      (pts
-        (xy 100 35) (xy 200 35) (xy 200 165) (xy 100 165)
-      )
-    )
-  )
-  (zone (net 1) (net_name GND) (layer F.Cu) (hatch edge 0.508)
-    (connect_pads (clearance 0.508))
-    (min_thickness 0.254)
-    (fill (arc_segments 16) (thermal_gap 0.508) (thermal_bridge_width 0.508))
-    (polygon
-      (pts
-        (xy 100 35) (xy 200 35) (xy 200 165) (xy 100 165)
-      )
-    )
-  )
 )

Commit message: v4 in production. i hate routing
Parts:
- moved R2 10.2 mm to (188.0, 132.1), turned to 270 degrees
Routing:
- net +5V: track 0.00 -> 290.2 mm, vias 0 -> 1
- net Net-(R9-Pad2): track 0.00 -> 162.7 mm
- net GND: track 0.00 -> 147.5 mm, vias 0 -> 5
- net Net-(C15-Pad2): track 0.00 -> 132.1 mm
- net /ANALOG_0: track 0.00 -> 127.6 mm
- net Net-(D5-Pad2): track 0.00 -> 121.5 mm
- net Net-(D6-Pad2): track 0.00 -> 120.2 mm
- net Net-(D4-Pad2): track 0.00 -> 117.3 mm
- net Net-(D3-Pad2): track 0.00 -> 113.2 mm
- net Net-(D2-Pad2): track 0.00 -> 113.1 mm
- net /DIGITAL_3: track 0.00 -> 108.3 mm, vias 0 -> 2
- net Net-(C10-Pad2): track 0.00 -> 100.6 mm
- net /DIGITAL_7: track 0.00 -> 82.6 mm
- net /ANALOG_1: track 0.00 -> 75.6 mm, vias 0 -> 1
- net Net-(C14-Pad1): track 0.00 -> 66.2 mm, vias 0 -> 1
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- added copper zone on B.Cu, net GND
- added copper zone on F.Cu, net GND
