File: pcb/drumkid v4/drumkid v3.sch (KiCad schematic (older format))
At the start: 53 parts, among them J1 Conn_01x04_Female, J5 Conn_01x05_Female, J6 Conn_01x04_Female, J7 Conn_01x06_Female, J8 Conn_01x05_Female, J9 AudioJack3_Ground_Switch, SW1 SW_SPDT, SW2 SW_Push, SW3 SW_Push, SW4 SW_Push, SW5 SW_Push, SW6 SW_Push, SW7 SW_Push, U2 ATmega328P-PU, U3 LM386, Y1 Crystal

Commit message: woah, did a bunch of stuff
Connections:
- net GND: now also C16.2, U3.4 (GND)
Changed lines of the file:
@@
 Connection ~ 7600 1900
 Wire Wire Line
-	7600 1900 8600 1900
+	7600 1900 7800 1900
 Wire Wire Line
 	6450 1050 6850 1050
@@
 	10000 4550 10150 4550
 Connection ~ 10700 4700
+Wire Wire Line
+	7800 1450 7800 1900
+Connection ~ 7800 1450
+Connection ~ 7800 1900
+Wire Wire Line
+	7800 1900 8600 1900
 $EndSCHEMATC
