File: pcb/drumkid v4/drumkid.sch (KiCad schematic (older format))
At the start: 53 parts, among them J1 Conn_01x04_Female, J5 Conn_01x05_Female, J6 Conn_01x04_Female, J7 Conn_01x06_Female, J8 Conn_01x05_Female, J9 AudioJack3_Ground_Switch, SW1 SW_SPDT, SW2 SW_Push, SW3 SW_Push, SW4 SW_Push, SW5 SW_Push, SW6 SW_Push, SW7 SW_Push, U2 ATmega328P-PU, U3 LM386, Y1 Crystal

Commit message: tidying up
Other:
- note added: "N.B. I left space for six decoupling capacitors\n(three for each pair of power/ground pins)\nbut final design only required C4 (100nF)"
- note added: "N.B. Pin 4 of LM386 needs to be\nmanually connected to ground\n(connection missing in PCB v4)"
Changed lines of the file:
@@
 EESchema Schematic File Version 4
-LIBS:drumkid v3-cache
+LIBS:drumkid-cache
 EELAYER 26 0
 EELAYER END
@@
 encoding utf-8
 Sheet 1 1
-Title ""
+Title "DrumKid"
 Date ""
-Rev ""
-Comp ""
+Rev "v4"
+Comp "by Matt Bradshaw"
 Comment1 ""
 Comment2 ""
@@
 Wire Wire Line
 	7800 1900 8600 1900
+Text Notes 7150 2200 0    50   ~ 0
+N.B. Pin 4 of LM386 needs to be\nmanually connected to ground\n(connection missing in PCB v4)
+Text Notes 600  4450 0    50   ~ 0
+N.B. I left space for six decoupling capacitors\n(three for each pair of power/ground pins)\nbut final design only required C4 (100nF)
 $EndSCHEMATC

Commit message: cleaned up repo for hackaday prize entry
Other:
- note added: "N.B. I left space for six decoupling capacitors\nin case they were needed (three for each pair\nof power/ground pins) but final design only\nrequired C4 (100nF)."
- note removed: "N.B. I left space for six decoupling capacitors\n(three for each pair of power/ground pins)\nbut final design only required C4 (100nF)"
Changed lines of the file:
@@
 N.B. Pin 4 of LM386 needs to be\nmanually connected to ground\n(connection missing in PCB v4)
 Text Notes 600  4450 0    50   ~ 0
-N.B. I left space for six decoupling capacitors\n(three for each pair of power/ground pins)\nbut final design only required C4 (100nF)
+N.B. I left space for six decoupling capacitors\nin case they were needed (three for each pair\nof power/ground pins) but final design only\nrequired C4 (100nF).
 $EndSCHEMATC
