File: pcb/drumkid v5/_saved_drumkid.sch (KiCad schematic (older format))
At the start: 62 parts, among them J1 Conn_01x02_Female, J2 DIN-5_180degree, J3 DIN-5_180degree, J5 Conn_01x05_Female, J6 Conn_01x04_Female, J7 Conn_01x06_Female, J8 Conn_01x05_Female, J9 AudioJack3_Ground_Switch, SW1 SW_SPDT, SW2 SW_Push, SW3 SW_Push, SW4 SW_Push, SW5 SW_Push, SW6 SW_Push, SW7 SW_Push, U1 6N138, U2 ATmega328P-PU, U3 LM386, Y1 Crystal

Commit message: more pcb progress
Parts:
- BT1: footprint Connector_PinHeader_2.54mm:PinHeader_1x02_P2.54mm_Vertical -> Connector_Wire:SolderWirePad_1x02_P5.08mm_Drill1.5mm
- gave numbers to parts that had none: 2
Connections:
- no-connect marks 8 -> 11
Changed lines of the file:
@@
 F 0 "BT1" H 4308 3446 50  0000 L CNN
 F 1 "Battery" H 4308 3355 50  0000 L CNN
-F 2 "Connector_PinHeader_2.54mm:PinHeader_1x02_P2.54mm_Vertical" V 4200 3460 50  0001 C CNN
+F 2 "Connector_Wire:SolderWirePad_1x02_P5.08mm_Drill1.5mm" V 4200 3460 50  0001 C CNN
 F 3 "~" V 4200 3460 50  0001 C CNN
 	1    4200 3400
@@
 	6800 5750 6800 4500
 $Comp
-L Device:LED D?
+L Device:LED D7
 U 1 1 5DBB8A3C
 P 6850 2500
-F 0 "D?" H 6842 2245 50  0000 C CNN
+F 0 "D7" H 6842 2245 50  0000 C CNN
 F 1 "LED" H 6842 2336 50  0000 C CNN
 F 2 "LED_THT:LED_D5.0mm" H 6850 2500 50  0001 C CNN
@@
 $EndComp
 $Comp
-L Device:R R?
+L Device:R R19
 U 1 1 5DBB8B2A
 P 6450 2500
-F 0 "R?" V 6243 2500 50  0000 C CNN
+F 0 "R19" V 6243 2500 50  0000 C CNN
 F 1 "220" V 6334 2500 50  0000 C CNN
 F 2 "Resistor_THT:R_Axial_DIN0207_L6.3mm_D2.5mm_P10.16mm_Horizontal" V 6380 2500 50  0001 C CNN
@@
 Wire Wire Line
 	6600 2500 6700 2500
+NoConn ~ 3100 7200
+NoConn ~ 3400 6900
+NoConn ~ 2800 6900
 $EndSCHEMATC
