File: pcb/drumkid v5/drumkid.kicad_pcb (KiCad board)
At the start: 2 copper layers, 90 x 140 mm, 70 parts, among them J1 Conn_01x02_Female, J2 DIN-5_180degree, J3 DIN-5_180degree, J5 Conn_01x05_Female, J6 Conn_01x04_Female, J7 Conn_01x06_Female, J8 Conn_01x05_Female, J9 AudioJack3_Ground_Switch, SW1 SW_SPDT, SW2 SW_Push, SW3 SW_Push, SW4 SW_Push, SW5 SW_Push, SW6 SW_Push, SW7 SW_Push, U1 6N138, U2 ATmega328P-PU, U3 LM386, Y1 Crystal

Commit message: adjusting silkscreen
Other:
- board text added: "BEAT TEMPO BEATS/BAR DRIFT"
- board text added: "CHANCE ZOOM RANGE MIDPOINT"
- board text added: "DROP DRONE_MOD DRONE_MIX DRONE_PITCH"
- board text added: "GO/STOP"
- board text added: "PITCH CRUSH CROP GLITCH"
- board text added: "SLOP SWING DELAY_TIME DELAY_MIX"
- board text removed: "A"
- board text removed: "B"
- board text removed: "C"
- board text removed: "X"
- board text removed: "Y"
- board text removed: "Z"
Changed lines of the file:
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@@
   )
   (gr_poly (pts (xy 78.5 99) (xy 98.5 99) (xy 98.5 94) (xy 78.5 94)) (layer F.SilkS) (width 0.15))
-  (gr_text Z (at 63.5 88.9) (layer B.SilkS)
-    (effects (font (size 1.5 1.5) (thickness 0.3)) (justify mirror))
+  (gr_text GO/STOP (at 68.58 88.9) (layer B.SilkS)
+    (effects (font (size 1.5 1.2) (thickness 0.3)) (justify left mirror))
   )
-  (gr_text Y (at 76.2 88.9) (layer B.SilkS)
-    (effects (font (size 1.5 1.5) (thickness 0.3)) (justify mirror))
+  (gr_text "DROP\nDRONE_MOD\nDRONE_MIX\nDRONE_PITCH" (at 81.28 92.71) (layer B.SilkS)
+    (effects (font (size 1.5 1.2) (thickness 0.3)) (justify left mirror))
   )
-  (gr_text X (at 88.9 88.9) (layer B.SilkS)
-    (effects (font (size 1.5 1.5) (thickness 0.3)) (justify mirror))
+  (gr_text "BEAT\nTEMPO\nBEATS/BAR\nDRIFT" (at 93.98 92.71) (layer B.SilkS)
+    (effects (font (size 1.5 1.2) (thickness 0.3)) (justify left mirror))
   )
-  (gr_text C (at 111.76 88.9) (layer B.SilkS)
-    (effects (font (size 1.5 1.5) (thickness 0.3)) (justify mirror))
+  (gr_text "SLOP\nSWING\nDELAY_TIME\nDELAY_MIX" (at 116.84 92.71) (layer B.SilkS)
+    (effects (font (size 1.5 1.2) (thickness 0.3)) (justify left mirror))
   )
-  (gr_text B (at 124.46 88.9) (layer B.SilkS)
-    (effects (font (size 1.5 1.5) (thickness 0.3)) (justify mirror))
+  (gr_text "PITCH\nCRUSH\nCROP\nGLITCH" (at 129.54 92.71) (layer B.SilkS)
+    (effects (font (size 1.5 1.2) (thickness 0.3)) (justify left mirror))
   )
-  (gr_text A (at 137.16 88.9) (layer B.SilkS)
-    (effects (font (size 1.5 1.5) (thickness 0.3)) (justify mirror))
+  (gr_text "CHANCE\nZOOM\nRANGE\nMIDPOINT" (at 142.24 92.71) (layer B.SilkS)
+    (effects (font (size 1.5 1.2) (thickness 0.3)) (justify left mirror))
   )
   (gr_text 1 (at 77 36) (layer B.SilkS)
