File: pcb/drumkid v5/drumkid.kicad_pcb (KiCad board)
At the start: 2 copper layers, 90 x 140 mm, 70 parts, among them J1 Conn_01x02_Female, J2 DIN-5_180degree, J3 DIN-5_180degree, J5 Conn_01x05_Female, J6 Conn_01x04_Female, J7 Conn_01x06_Female, J8 Conn_01x05_Female, J9 AudioJack3_Ground_Switch, SW1 SW_SPDT, SW2 SW_Push, SW3 SW_Push, SW4 SW_Push, SW5 SW_Push, SW6 SW_Push, SW7 SW_Push, U1 6N138, U2 ATmega328P-PU, U3 LM386, Y1 Crystal

Commit message: v5 gerbers and MIDI input code
Other:
- board text added: "A"
- board text added: "B"
- board text added: "C"
- board text added: "X"
- board text added: "Y"
- board text added: "Z"
Changed lines of the file:
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@@
   (general
     (thickness 1.6)
-    (drawings 43)
+    (drawings 49)
     (tracks 427)
     (zones 0)
@@
       (outputformat 1)
       (mirror false)
-      (drillshape 1)
+      (drillshape 0)
       (scaleselection 1)
-      (outputdirectory ""))
+      (outputdirectory "gerbers/"))
   )
   (net 0 "")
@@
     )
   )
+  (gr_text Z (at 63.5 71.12) (layer B.SilkS)
+    (effects (font (size 1.5 1.5) (thickness 0.3)) (justify mirror))
+  )
+  (gr_text Y (at 76.2 71.12) (layer B.SilkS)
+    (effects (font (size 1.5 1.5) (thickness 0.3)) (justify mirror))
+  )
+  (gr_text X (at 88.9 71.12) (layer B.SilkS)
+    (effects (font (size 1.5 1.5) (thickness 0.3)) (justify mirror))
+  )
+  (gr_text C (at 111.76 71.12) (layer B.SilkS)
+    (effects (font (size 1.5 1.5) (thickness 0.3)) (justify mirror))
+  )
+  (gr_text B (at 124.46 71.12) (layer B.SilkS)
+    (effects (font (size 1.5 1.5) (thickness 0.3)) (justify mirror))
+  )
+  (gr_text A (at 137.16 71.12) (layer B.SilkS)
+    (effects (font (size 1.5 1.5) (thickness 0.3)) (justify mirror))
+  )
   (gr_text "DrumKid v05\nby Matt Bradshaw\nmattbradshawdesign.com" (at 101 95.5) (layer F.SilkS)
     (effects (font (size 1.5 1.5) (thickness 0.3)) (justify left))
@@
   )
   (gr_poly (pts (xy 78.5 99) (xy 98.5 99) (xy 98.5 94) (xy 78.5 94)) (layer F.SilkS) (width 0.15))
-  (gr_text GO/STOP (at 68.58 88.9) (layer B.SilkS)
+  (gr_text GO/STOP (at 68.58 89.535) (layer B.SilkS)
     (effects (font (size 1.5 1.2) (thickness 0.3)) (justify left mirror))
   )
-  (gr_text "DROP\nDRONE_MOD\nDRONE_MIX\nDRONE_PITCH" (at 81.28 92.71) (layer B.SilkS)
+  (gr_text "DROP\nDRONE_MOD\nDRONE_MIX\nDRONE_PITCH" (at 81.28 93.345) (layer B.SilkS)
     (effects (font (size 1.5 1.2) (thickness 0.3)) (justify left mirror))
   )
-  (gr_text "BEAT\nTEMPO\nBEATS/BAR\nDRIFT" (at 93.98 92.71) (layer B.SilkS)
+  (gr_text "BEAT\nTEMPO\nBEATS/BAR\nDRIFT" (at 93.98 93.345) (layer B.SilkS)
     (effects (font (size 1.5 1.2) (thickness 0.3)) (justify left mirror))
   )
-  (gr_text "SLOP\nSWING\nDELAY_TIME\nDELAY_MIX" (at 116.84 92.71) (layer B.SilkS)
+  (gr_text "SLOP\nSWING\nDELAY_TIME\nDELAY_MIX" (at 116.84 93.345) (layer B.SilkS)
     (effects (font (size 1.5 1.2) (thickness 0.3)) (justify left mirror))
   )
-  (gr_text "PITCH\nCRUSH\nCROP\nGLITCH" (at 129.54 92.71) (layer B.SilkS)
+  (gr_text "PITCH\nCRUSH\nCROP\nGLITCH" (at 129.54 93.345) (layer B.SilkS)
     (effects (font (size 1.5 1.2) (thickness 0.3)) (justify left mirror))
   )
-  (gr_text "CHANCE\nZOOM\nRANGE\nMIDPOINT" (at 142.24 92.71) (layer B.SilkS)
+  (gr_text "CHANCE\nZOOM\nRANGE\nMIDPOINT" (at 142.24 93.345) (layer B.SilkS)
     (effects (font (size 1.5 1.2) (thickness 0.3)) (justify left mirror))
   )
