File: v6/pcb/drumkid.kicad_pcb (KiCad board)
At the start: 2 copper layers, 90 x 140 mm, 70 parts, among them J1 Conn_01x02_Female, J2 DIN-5_180degree, J3 DIN-5_180degree, J5 Conn_01x05_Female, J6 Conn_01x04_Female, J7 Conn_01x06_Female, J8 Conn_01x05_Female, J9 AudioJack3_Ground_Switch, SW1 SW_SPDT, SW2 SW_Push, SW3 SW_Push, SW4 SW_Push, SW5 SW_Push, SW6 SW_Push, SW7 SW_Push, U1 6N138, U2 ATmega328P-PU, U3 LM386, Y1 Crystal

Commit message: nearly all V4 params now working in V6
Other:
- board text added: "CHANCE ZOOM MIDPOINT RANGE"
- board text removed: "CHANCE ZOOM RANGE MIDPOINT"
Changed lines of the file:
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@@
   (page A4)
   (layers
-    (0 F.Cu signal)
-    (31 B.Cu signal)
+    (0 F.Cu signal hide)
+    (31 B.Cu signal hide)
     (32 B.Adhes user)
     (33 F.Adhes user)
@@
     (effects (font (size 1.5 1.2) (thickness 0.3)) (justify left mirror))
   )
-  (gr_text "CHANCE\nZOOM\nRANGE\nMIDPOINT" (at 142.24 93.345) (layer B.SilkS)
+  (gr_text "CHANCE\nZOOM\nMIDPOINT\nRANGE" (at 142.24 93.345) (layer B.SilkS)
     (effects (font (size 1.5 1.2) (thickness 0.3)) (justify left mirror))
   )

Commit message: the zoom function is weird and confusing
Other:
- board text added: "+ -"
- board text added: "???? DRONE_MOD DRONE_MIX DRONE_PITCH"
- board text added: "BEAT TEMPO BEATS/BAR DROP"
- board text added: "DrumKid v06 by Matt Bradshaw mattbradshawdesign.com github.com/mattybrad/drumkid"
- board text added: "SLOP SWING DELAY GREMLIN"
- board text added: "drumkid"
- board text added: "hackable aleatoric lo-fi drum machine"
- board text removed: "BEAT TEMPO BEATS/BAR DRIFT"
- board text removed: "DROP DRONE_MOD DRONE_MIX DRONE_PITCH"
- board text removed: "DrumKid v05 by Matt Bradshaw mattbradshawdesign.com"
- board text removed: "SLOP SWING DELAY_TIME DELAY_MIX"
- board text removed: "d"
- board text removed: "k"
Changed lines of the file:
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@@
   (general
     (thickness 1.6)
-    (drawings 49)
+    (drawings 44)
     (tracks 427)
     (zones 0)
@@
     (35 F.Paste user)
     (36 B.SilkS user)
-    (37 F.SilkS user)
+    (37 F.SilkS user hide)
     (38 B.Mask user)
     (39 F.Mask user)
@@
     (tags connector)
     (attr virtual)
-    (fp_text reference BT1 (at 2.54 -3.81) (layer F.SilkS)
+    (fp_text reference BT1 (at 2.88 2.32) (layer F.SilkS)
       (effects (font (size 1 1) (thickness 0.15)))
     )
@@
     )
   )
+  (gr_text "+   -" (at 73.66 103) (layer F.SilkS)
+    (effects (font (size 1.5 1.5) (thickness 0.3)))
+  )
+  (gr_text drumkid (at 100.33 59.69) (layer B.SilkS)
+    (effects (font (size 3.6 3.6) (thickness 0.6)) (justify mirror))
+  )
+  (gr_text "hackable aleatoric\nlo-fi drum machine" (at 111 65) (layer B.SilkS)
+    (effects (font (size 1.4 1.4) (thickness 0.3)) (justify left mirror))
+  )
   (gr_text Z (at 63.5 71.12) (layer B.SilkS)
     (effects (font (size 1.5 1.5) (thickness 0.3)) (justify mirror))
@@
     (effects (font (size 1.5 1.5) (thickness 0.3)) (justify mirror))
   )
-  (gr_text "DrumKid v05\nby Matt Bradshaw\nmattbradshawdesign.com" (at 101 95.5) (layer F.SilkS)
+  (gr_text "DrumKid v06\nby Matt Bradshaw\nmattbradshawdesign.com\ngithub.com/mattybrad/drumkid" (at 95 97) (layer F.SilkS)
     (effects (font (size 1.5 1.5) (thickness 0.3)) (justify left))
   )
-  (gr_text d (at 102.8 63.1) (layer B.SilkS)
-    (effects (font (size 10 10) (thickness 0.3)) (justify mirror))
-  )
-  (gr_text k (at 96.5 62.9) (layer B.SilkS)
-    (effects (font (size 10 10) (thickness 0.3)) (justify mirror))
-  )
-  (gr_text k (at 96.7 62.6) (layer B.SilkS)
-    (effects (font (size 10 10) (thickness 0.3)) (justify mirror))
-  )
-  (gr_text k (at 96.3 62.1) (layer B.SilkS)
-    (effects (font (size 10 10) (thickness 0.3)) (justify mirror))
-  )
-  (gr_text d (at 103.4 63.6) (layer B.SilkS)
-    (effects (font (size 10 10) (thickness 0.3)) (justify mirror))
-  )
-  (gr_text d (at 103 62.9) (layer B.SilkS)
-    (effects (font (size 10 10) (thickness 0.3)) (justify mirror))
-  )
-  (gr_text k (at 97.1 62.8) (layer B.SilkS)
-    (effects (font (size 10 10) (thickness 0.3)) (justify mirror))
-  )
-  (gr_text d (at 102.7 62.5) (layer B.SilkS)
-    (effects (font (size 10 10) (thickness 0.3)) (justify mirror))
-  )
   (gr_text "8\n7\n6\n5\n\n\nGND\nVCC\n4\n3\n2\n1\n0" (at 88.9 128.27 270) (layer F.SilkS)
     (effects (font (size 1.5 1.5) (thickness 0.3)) (justify left))
@@
   (gr_line (start 145 35) (end 145 140) (layer Edge.Cuts) (width 0.2))
   (gr_arc (start 60 35) (end 60 30) (angle -90) (layer Edge.Cuts) (width 0.2))
-  (gr_text "SERIAL NUMBER" (at 88.5 93) (layer F.SilkS)
+  (gr_text "SERIAL NUMBER" (at 82 94) (layer F.SilkS)
     (effects (font (size 1.5 1.5) (thickness 0.3)))
   )
-  (gr_poly (pts (xy 78.5 99) (xy 98.5 99) (xy 98.5 94) (xy 78.5 94)) (layer F.SilkS) (width 0.15))
+  (gr_poly (pts (xy 72 101) (xy 92 101) (xy 92 96) (xy 72 96)) (layer F.SilkS) (width 0.15))
   (gr_text GO/STOP (at 68.58 89.535) (layer B.SilkS)
     (effects (font (size 1.5 1.2) (thickness 0.3)) (justify left mirror))
   )
-  (gr_text "DROP\nDRONE_MOD\nDRONE_MIX\nDRONE_PITCH" (at 81.28 93.345) (layer B.SilkS)
+  (gr_text "????\nDRONE_MOD\nDRONE_MIX\nDRONE_PITCH" (at 81.28 93.345) (layer B.SilkS)
     (effects (font (size 1.5 1.2) (thickness 0.3)) (justify left mirror))
   )
-  (gr_text "BEAT\nTEMPO\nBEATS/BAR\nDRIFT" (at 93.98 93.345) (layer B.SilkS)
+  (gr_text "BEAT\nTEMPO\nBEATS/BAR\nDROP" (at 93.98 93.345) (layer B.SilkS)
     (effects (font (size 1.5 1.2) (thickness 0.3)) (justify left mirror))
   )
-  (gr_text "SLOP\nSWING\nDELAY_TIME\nDELAY_MIX" (at 116.84 93.345) (layer B.SilkS)
+  (gr_text "SLOP\nSWING\nDELAY\nGREMLIN" (at 116.84 93.345) (layer B.SilkS)
     (effects (font (size 1.5 1.2) (thickness 0.3)) (justify left mirror))
   )

Commit message: half way through pcb layout v6
Parts:
- removed C10: 220uF, drumkidcustom:CP_Radial_D6.3mm_P2.50mm
- removed C16, C18: 100nF, drumkidcustom:C_Disc_D3.4mm_W2.1mm_P2.50mm
- removed C17: 10uF, drumkidcustom:CP_Radial_D6.3mm_P2.50mm
- removed C5, C6: 22pF, drumkidcustom:C_Disc_D3.4mm_W2.1mm_P2.50mm
- removed C7: 220nF, drumkidcustom:C_Disc_D3.4mm_W2.1mm_P2.50mm
- removed J5, J8: Conn_01x05_Female, Connector_PinHeader_2.54mm:PinHeader_1x05_P2.54mm_Vertical
- removed J6: Conn_01x04_Female, Connector_PinHeader_2.54mm:PinHeader_1x04_P2.54mm_Vertical
- removed J7: Conn_01x06_Female, Connector_PinHeader_2.54mm:PinHeader_1x06_P2.54mm_Vertical
- removed R12: 680, drumkidcustom:R_Axial_DIN0207_L6.3mm_D2.5mm_P10.16mm_Horizontal
- removed R13: 330, drumkidcustom:R_Axial_DIN0207_L6.3mm_D2.5mm_P10.16mm_Horizontal
- removed R14, R16, R18, R19: 220, drumkidcustom:R_Axial_DIN0207_L6.3mm_D2.5mm_P10.16mm_Horizontal
- removed R15: 10k, drumkidcustom:R_Axial_DIN0207_L6.3mm_D2.5mm_P10.16mm_Horizontal
- removed R17: 470, drumkidcustom:R_Axial_DIN0207_L6.3mm_D2.5mm_P10.16mm_Horizontal
- removed U2: ATmega328P-PU, Package_DIP:DIP-28_W7.62mm_Socket
- removed U3: LM386, Package_DIP:DIP-8_W7.62mm_Socket
- removed Y1: Crystal, Crystal:Crystal_HC49-4H_Vertical
- added A1: Arduino_Nano_v3.x, Module:Arduino_Nano_WithMountingHoles, F.Cu at (101.1, 118.9)
- added D8: 1N5817, Diode_THT:D_DO-41_SOD81_P10.16mm_Horizontal, F.Cu at (47.6, 93.4)
- added J4: Conn_01x15, Connector_PinSocket_2.54mm:PinSocket_1x15_P2.54mm_Vertical, F.Cu at (65.5, 116.4)
- added SW8: SW_SPDT, drumkidcustom:EG1206, F.Cu at (55.0, 185.0)
- C1: value 220nF -> CP; footprint drumkidcustom:C_Disc_D3.4mm_W2.1mm_P2.50mm -> Capacitor_THT:CP_Radial_D6.3mm_P2.50mm
- C2: value 220nF -> C; footprint drumkidcustom:C_Disc_D3.4mm_W2.1mm_P2.50mm -> Capacitor_THT:C_Disc_D3.4mm_W2.1mm_P2.50mm
- C3: value 1nF -> CP; footprint drumkidcustom:C_Disc_D3.4mm_W2.1mm_P2.50mm -> Capacitor_THT:CP_Radial_D6.3mm_P2.50mm
- C4: value 100nF -> C; footprint drumkidcustom:C_Disc_D3.4mm_W2.1mm_P2.50mm -> Capacitor_THT:C_Disc_D3.4mm_W2.1mm_P2.50mm
- D1: value 1N4148 -> LED; footprint Diode_THT:D_DO-35_SOD27_P7.62mm_Horizontal -> drumkidcustom:LED_D5.0mm; moved to B.Cu
- D7: value LED -> 1N4148; footprint drumkidcustom:LED_D5.0mm -> Diode_THT:D_DO-35_SOD27_P7.62mm_Horizontal
- J1: value Conn_01x02_Female -> DIN-5_180degree; footprint Connector_PinHeader_2.54mm:PinHeader_1x02_P2.54mm_Vertical -> drumkidcustom:MIDI_DIN5
- J3: value DIN-5_180degree -> Conn_01x15; footprint drumkidcustom:MIDI_DIN5 -> Connector_PinSocket_2.54mm:PinSocket_1x15_P2.54mm_Vertical
- R1, R3, R4, R5, R6: value 220 -> 470
- R11: value 10 -> 220
- R2: value 10k -> 470
- R8: value 680 -> 10k
- R9: value 4.7k -> 470
- RV1: value 10k -> R_POT
- RV5: value R_POT -> 10k
- SW1: value SW_SPDT -> SW_Push; footprint drumkidcustom:EG1206 -> drumkidcustom:SW_PUSH-12mm_Wuerth-430476085716
- SW7: value SW_Push -> SW_SPDT; footprint drumkidcustom:SW_PUSH-12mm_Wuerth-430476085716 -> drumkidcustom:EG1206
- moved D7 97.7 mm to (157.5, 91.4)
- moved R1 93.7 mm to (175.0, 108.0)
- moved D1 87.2 mm to (129.0, 50.0)
- moved C3 85.1 mm to (201.8, 123.4)
- moved R10 85.1 mm to (199.3, 136.1)
- moved R2 85.1 mm to (153.6, 128.5)
- moved R5 85.1 mm to (163.7, 146.2)
- moved R9 85.1 mm to (209.5, 123.4)
- moved C1 85.1 mm to (201.8, 118.3)
- moved C2 85.1 mm to (204.4, 136.1)
- moved C4 85.1 mm to (173.9, 118.3)
- moved R11 85.1 mm to (214.5, 113.2)
- moved R3 85.1 mm to (158.7, 146.2)
- moved R6 85.1 mm to (176.4, 146.2)
- moved R8 85.1 mm to (212.0, 123.4)
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Connections:
- C1 pad 1: Net-(C1-Pad1) -> VCC
- C2 pad 1: Net-(C1-Pad1) -> VCC
- C2 pad 2: Net-(C2-Pad2) -> GND
- C3 pad 1: Net-(C3-Pad1) -> VCC
- C4 pad 1: +5V -> VCC
- D1 pad 1: Net-(D1-Pad1) -> GND
- D7 pad 1: GND -> Net-(D7-Pad1)
- J1 pad 1: +5V -> Net-(J1-Pad1)
- J1 pad 2: GND -> Net-(J1-Pad2)
- J2 pad 2: Net-(J2-Pad2) -> GND
- J2 pad 5: Net-(D1-Pad2) -> Net-(J2-Pad5)
- J3 pad 1: Net-(J3-Pad1) -> /DIGITAL_13
- J3 pad 2: GND -> /3V3
- J3 pad 3: Net-(J3-Pad3) -> /AREF
- J3 pad 4: Net-(J3-Pad4) -> /ANALOG_0
- J3 pad 5: Net-(J3-Pad5) -> /ANALOG_1
- J9 pad R: Net-(C10-Pad2) -> Net-(J9-PadR)
- J9 pad T: Net-(C10-Pad2) -> Net-(J9-PadR)
- R1 pad 1: Net-(C1-Pad1) -> Net-(D1-Pad2)
- R1 pad 2: /DIGITAL_9 -> VCC
- R10 pad 1: Net-(R10-Pad1) -> Net-(J2-Pad5)
- R10 pad 2: GND -> /DIGITAL_1
- R11 pad 1: Net-(C18-Pad2) -> Net-(J2-Pad4)
- R11 pad 2: GND -> VCC
- R2 pad 1: Net-(R2-Pad1) -> Net-(D2-Pad2)
- R2 pad 2: +5V -> /DIGITAL_2
- R3 pad 1: Net-(D2-Pad2) -> Net-(D3-Pad2)
- R3 pad 2: /DIGITAL_2 -> /DIGITAL_3
- R4 pad 1: Net-(D3-Pad2) -> Net-(D4-Pad2)
- R4 pad 2: /DIGITAL_3 -> /DIGITAL_11
- R5 pad 1: Net-(D4-Pad2) -> Net-(D5-Pad2)
- R5 pad 2: /DIGITAL_4 -> /DIGITAL_12
- R6 pad 1: Net-(D5-Pad2) -> Net-(D6-Pad2)
- R6 pad 2: /DIGITAL_5 -> /DIGITAL_13
- R7 pad 1: Net-(D6-Pad2) -> Net-(D7-Pad1)
- R7 pad 2: /DIGITAL_6 -> Net-(J1-Pad4)
- R8 pad 1: Net-(C3-Pad1) -> GND
- R8 pad 2: Net-(C1-Pad1) -> Net-(R8-Pad2)
- R9 pad 1: Net-(R10-Pad1) -> VCC
- RV1 pad 1: Net-(C7-Pad1) -> VCC
- RV1 pad 2: Net-(R9-Pad2) -> /ANALOG_0
- RV2 pad 1: +5V -> VCC
- RV2 pad 2: /ANALOG_0 -> /ANALOG_1
- RV3 pad 1: +5V -> VCC
- RV3 pad 2: /ANALOG_1 -> /ANALOG_2
- RV4 pad 1: +5V -> VCC
- RV4 pad 2: /ANALOG_2 -> /ANALOG_3
- RV5 pad 1: +5V -> /DIGITAL_9
- RV5 pad 2: /ANALOG_3 -> Net-(J9-PadR)
- SW1 pad 1: +5V -> /DIGITAL_4
- SW1 pad 2: Net-(BT1-Pad1) -> GND
- SW2 pad 1: /DIGITAL_7 -> /DIGITAL_5
- SW3 pad 1: /DIGITAL_8 -> /DIGITAL_6
- SW4 pad 1: /DIGITAL_10 -> /DIGITAL_7
- SW5 pad 1: /DIGITAL_11 -> /DIGITAL_8
- SW6 pad 1: /DIGITAL_12 -> /DIGITAL_10
- SW7 pad 1: /DIGITAL_13 -> Net-(SW7-Pad1)
- SW7 pad 2: GND -> Net-(BT1-Pad1)
- U1 pad 2: Net-(D1-Pad1) -> Net-(D7-Pad1)
- U1 pad 3: Net-(D1-Pad2) -> Net-(D7-Pad2)
- U1 pad 6: /DIGITAL_0 -> Net-(R9-Pad2)
- U1 pad 7: Net-(R15-Pad2) -> Net-(R8-Pad2)
- U1 pad 8: +5V -> VCC
Routing:
- net +5V: track 295.7 -> 0.00 mm
- net GND: track 268.4 -> 0.00 mm, vias 4 -> 0
- net Net-(D4-Pad2): track 184.2 -> 0.00 mm
- net Net-(D5-Pad2): track 162.1 -> 0.00 mm
- net Net-(D3-Pad2): track 139.0 -> 0.00 mm
- net Net-(D6-Pad2): track 136.2 -> 0.00 mm
- net /ANALOG_1: track 127.4 -> 0.00 mm
- net Net-(D2-Pad2): track 114.7 -> 0.00 mm
- net Net-(C7-Pad1): track 110.1 -> 0.00 mm
- net /ANALOG_0: track 99.0 -> 0.00 mm
- net Net-(BT1-Pad1): track 92.1 -> 0.00 mm
- net Net-(C10-Pad2): track 88.4 -> 0.00 mm
- net /DIGITAL_7: track 86.5 -> 0.00 mm, vias 2 -> 0
- net /DIGITAL_13: track 82.1 -> 0.00 mm
- net Net-(R9-Pad2): track 81.2 -> 0.00 mm
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- removed copper zone on B.Cu, net GND
- removed copper zone on F.Cu, net GND

Commit message: some decent pcb progress
Parts:
- moved R11 139.4 mm to (78.7, 144.8), turned to 0 degrees
- moved R10 121.1 mm to (78.7, 147.3), turned to 0 degrees
- moved C1 111.1 mm to (94.0, 144.8)
- moved C3 108.2 mm to (94.0, 114.3)
- moved C2 103.4 mm to (101.6, 147.3), turned to 90 degrees
- moved R6 101.7 mm to (83.8, 104.1), turned to 270 degrees
- moved U1 93.2 mm to (121.9, 119.4)
- moved R5 88.1 mm to (86.4, 104.1), turned to 270 degrees
- moved R4 83.7 mm to (88.9, 104.1), turned to 270 degrees
- moved SW8 83.5 mm to (129.5, 147.3), turned to 90 degrees
- moved C4 80.8 mm to (94.0, 106.7), turned to 0 degrees
- moved R8 75.1 mm to (137.2, 129.5)
- moved R9 74.9 mm to (134.6, 119.4), turned to 270 degrees
- moved R7 72.3 mm to (106.7, 147.3), turned to 0 degrees
- moved D8 71.5 mm to (109.2, 129.5), turned to 90 degrees
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Connections:
- A1 pad 27: Net-(A1-Pad27) -> VCC
- D8 pad 1: Net-(A1-Pad27) -> VCC
- D8 pad 2: VCC -> Net-(D8-Pad2)
- SW7 pad 3: VCC -> Net-(D8-Pad2)
Other:
- board text removed: "8 7 6 5 GND VCC 4 3 2 1 0"
- board text removed: "9 10 11 12 13 A0 A1 A2 A3 A4 A5"

Commit message: more pcb layout
Parts:
- D7, SW7: moved to F.Cu
- moved SW1 7.62 mm to (134.6, 81.3)
- moved SW2 7.62 mm to (121.9, 81.3)
- moved SW3 7.62 mm to (109.2, 81.3)
- moved SW4 7.62 mm to (86.4, 81.3)
- moved SW5 7.62 mm to (73.7, 81.3)
- moved SW6 7.62 mm to (61.0, 81.3)
- moved SW7 6.03 mm to (85.0, 40.0), turned to 180 degrees
Other:
- board text added: "Arduino Nano 3"
- board text added: "D"
- board text added: "USB port this end"
- board text added: "chance pitch slop beat"
- board text added: "start/stop"
- board text added: "tap tempo"
- board text removed: "???? DRONE_MOD DRONE_MIX DRONE_PITCH"
- board text removed: "BEAT TEMPO BEATS/BAR DROP"
- board text removed: "CHANCE ZOOM MIDPOINT RANGE"
- board text removed: "GO/STOP"
- board text removed: "PITCH CRUSH CROP GLITCH"
- board text removed: "SLOP SWING DELAY GREMLIN"
- board text removed: "X"
- board text removed: "Y"
- board text removed: "Z"

Commit message: about to start routing
Other:
- board text added: "arduino"
- board text added: "midi"
Changed lines of the file:
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@@
   (general
     (thickness 1.6)
-    (drawings 46)
+    (drawings 48)
     (tracks 0)
     (zones 0)
@@
     )
   )
+  (gr_text arduino (at 133.35 138.43) (layer F.SilkS)
+    (effects (font (size 1.2 1.2) (thickness 0.3)) (justify left))
+  )
+  (gr_text midi (at 133.35 149.86) (layer F.SilkS)
+    (effects (font (size 1.2 1.2) (thickness 0.3)) (justify left))
+  )
   (gr_line (start 144.9324 77.47) (end 54.991 77.47) (layer B.SilkS) (width 0.1))

Commit message: routing half done
Routing:
- net /ANALOG_1: track 0.00 -> 176.5 mm
- net /ANALOG_0: track 0.00 -> 166.9 mm
- net VCC: track 0.00 -> 122.4 mm
- net Net-(D8-Pad2): track 0.00 -> 101.3 mm
- net /DIGITAL_9: track 0.00 -> 96.4 mm
- net Net-(BT1-Pad1): track 0.00 -> 85.9 mm
- net /DIGITAL_4: track 0.00 -> 85.3 mm
- net /ANALOG_3: track 0.00 -> 83.5 mm
- net /DIGITAL_5: track 0.00 -> 75.7 mm, vias 0 -> 1
- net /ANALOG_2: track 0.00 -> 73.2 mm
- net /DIGITAL_6: track 0.00 -> 64.2 mm, vias 0 -> 2
- net Net-(D6-Pad2): track 0.00 -> 60.9 mm
- net Net-(D5-Pad2): track 0.00 -> 57.5 mm
- net Net-(D4-Pad2): track 0.00 -> 56.4 mm
- net GND: track 0.00 -> 55.3 mm
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