File: v6/pcb/drumkid.kicad_pcb (KiCad board)
At the start: 2 copper layers, 90 x 140 mm, 52 parts, among them J1 DIN-5_180degree, J2 DIN-5_180degree, J3 Conn_01x15, J4 Conn_01x15, J9 AudioJack3_Ground_Switch, SW1 SW_Push, SW2 SW_Push, SW3 SW_Push, SW4 SW_Push, SW5 SW_Push, SW6 SW_Push, SW7 SW_SPDT, SW8 SW_SPDT, U1 6N138

Commit message: routing done?
Routing:
- net VCC: track 122.4 -> 256.7 mm, vias 0 -> 2
- net Net-(D3-Pad2): track 0.00 -> 111.9 mm
- net Net-(D2-Pad2): track 0.00 -> 101.2 mm
- net Net-(D1-Pad2): track 0.00 -> 89.0 mm
- net /RESET: track 2.54 -> 21.6 mm, vias 0 -> 1
- added copper zone on B.Cu, net GND
- added copper zone on F.Cu, net GND
Other:
- board text added: "a"
- board text added: "aleatoric drum machine"
- board text added: "b"
- board text added: "c"
- board text added: "d"
- board text added: "midi in"
- board text added: "midi out"
- board text removed: "A"
- board text removed: "B"
- board text removed: "C"
- board text removed: "D"
- board text removed: "MIDI IN"
- board text removed: "MIDI OUT"
- board text removed: "hackable aleatoric lo-fi drum machine"
Changed lines of the file:
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@@
     (thickness 1.6)
     (drawings 48)
-    (tracks 247)
+    (tracks 293)
     (zones 0)
     (modules 52)
@@
     (effects (font (size 3.6 3.6) (thickness 0.6)) (justify mirror))
   )
-  (gr_text "hackable aleatoric\nlo-fi drum machine" (at 111 65) (layer B.SilkS)
-    (effects (font (size 1.4 1.4) (thickness 0.3)) (justify left mirror))
+  (gr_text "aleatoric drum machine" (at 100.5 64) (layer B.SilkS)
+    (effects (font (size 1.2 1.2) (thickness 0.3)) (justify mirror))
   )
   (gr_text "tap tempo" (at 63.5 97.12) (layer B.SilkS)
     (effects (font (size 1.5 1.5) (thickness 0.3)) (justify mirror))
   )
-  (gr_text D (at 76.2 97.12) (layer B.SilkS)
+  (gr_text d (at 76.2 97.12) (layer B.SilkS)
     (effects (font (size 1.5 1.5) (thickness 0.3)) (justify mirror))
   )
-  (gr_text C (at 88.9 97.12) (layer B.SilkS)
+  (gr_text c (at 88.9 97.12) (layer B.SilkS)
     (effects (font (size 1.5 1.5) (thickness 0.3)) (justify mirror))
   )
-  (gr_text B (at 111.76 97.12) (layer B.SilkS)
+  (gr_text b (at 111.76 97.12) (layer B.SilkS)
     (effects (font (size 1.5 1.5) (thickness 0.3)) (justify mirror))
   )
-  (gr_text A (at 124.46 97.12) (layer B.SilkS)
+  (gr_text a (at 124.46 97.12) (layer B.SilkS)
     (effects (font (size 1.5 1.5) (thickness 0.3)) (justify mirror))
   )
@@
   (gr_circle (center 100 50) (end 102.5 50) (layer F.SilkS) (width 0.2))
   (gr_circle (center 100 80) (end 100 77.5) (layer F.SilkS) (width 0.2))
-  (gr_text "MIDI OUT" (at 88.9 167.64) (layer B.SilkS)
+  (gr_text "midi out" (at 88.9 167.64) (layer B.SilkS)
     (effects (font (size 1.5 1.5) (thickness 0.3)) (justify mirror))
   )
-  (gr_text "MIDI IN" (at 111.76 167.64) (layer B.SilkS)
+  (gr_text "midi in" (at 111.76 167.64) (layer B.SilkS)
     (effects (font (size 1.5 1.5) (thickness 0.3)) (justify mirror))
   )
@@
   (segment (start 92.71 118.11) (end 91.44 119.38) (width 0.25) (layer F.Cu) (net 15))
   (segment (start 100.33 118.11) (end 92.71 118.11) (width 0.25) (layer F.Cu) (net 15))
+  (segment (start 104.14 104.14) (end 104.14 102.87) (width 0.25) (layer B.Cu) (net 16))
+  (segment (start 141.75501 60.292598) (end 137.342412 55.88) (width 0.25) (layer B.Cu) (net 16))
+  (segment (start 141.755011 94.758799) (end 141.75501 60.292598) (width 0.25) (layer B.Cu) (net 16))
+  (segment (start 137.823791 98.690019) (end 141.755011 94.758799) (width 0.25) (layer B.Cu) (net 16))
+  (segment (start 104.14 102.87) (end 108.31998 98.69002) (width 0.25) (layer B.Cu) (net 16))
+  (segment (start 108.31998 98.69002) (end 137.823791 98.690019) (width 0.25) (layer B.Cu) (net 16))
+  (segment (start 127.42 55.88) (end 121.54 50) (width 0.25) (layer B.Cu) (net 16))
+  (segment (start 137.342412 55.88) (end 127.42 55.88) (width 0.25) (layer B.Cu) (net 16))
+  (segment (start 141.305001 60.478999) (end 137.976002 57.15) (width 0.25) (layer B.Cu) (net 17))
+  (segment (start 141.305001 94.572399) (end 141.305001 60.478999) (width 0.25) (layer B.Cu) (net 17))
+  (segment (start 137.63739 98.24001) (end 141.305001 94.572399) (width 0.25) (layer B.Cu) (net 17))
+  (segment (start 101.6 104.14) (end 107.49999 98.24001) (width 0.25) (layer B.Cu) (net 17))
+  (segment (start 107.49999 98.24001) (end 137.63739 98.24001) (width 0.25) (layer B.Cu) (net 17))
+  (segment (start 118.69 57.15) (end 111.54 50) (width 0.25) (layer B.Cu) (net 17))
+  (segment (start 137.976002 57.15) (end 118.69 57.15) (width 0.25) (layer B.Cu) (net 17))
   (segment (start 88.9 119.38) (end 88.9 121.92) (width 0.25) (layer F.Cu) (net 18))
   (via (at 99.06 116.84) (size 0.8) (drill 0.4) (layers F.Cu B.Cu) (net 18))
@@
   (segment (start 82.405001 148.445001) (end 90.276461 148.445001) (width 0.25) (layer F.Cu) (net 31))
   (segment (start 78.74 144.78) (end 82.405001 148.445001) (width 0.25) (layer F.Cu) (net 31))
+  (segment (start 106.68 104.14) (end 110.49 100.33) (width 0.25) (layer B.Cu) (net 33))
+  (segment (start 132.439999 50.899999) (end 131.54 50) (width 0.25) (layer B.Cu) (net 33))
+  (segment (start 132.998821 50.899999) (end 132.439999 50.899999) (width 0.25) (layer B.Cu) (net 33))
+  (segment (start 142.205019 60.106197) (end 132.998821 50.899999) (width 0.25) (layer B.Cu) (net 33))
+  (segment (start 142.20502 94.945198) (end 142.205019 60.106197) (width 0.25) (layer B.Cu) (net 33))
+  (segment (start 136.820218 100.33) (end 142.20502 94.945198) (width 0.25) (layer B.Cu) (net 33))
+  (segment (start 110.49 100.33) (end 136.820218 100.33) (width 0.25) (layer B.Cu) (net 33))
   (segment (start 119.38 127) (end 121.92 124.46) (width 0.25) (layer F.Cu) (net 37))
   (segment (start 116.84 127) (end 119.38 127) (width 0.25) (layer F.Cu) (net 37))
@@
   (segment (start 106.68 114.3) (end 106.68 123.19) (width 0.625) (layer F.Cu) (net 39))
   (segment (start 106.68 123.19) (end 106.68 118.11) (width 0.625) (layer F.Cu) (net 39))
+  (segment (start 64.399999 67.680001) (end 63.5 68.58) (width 0.625) (layer F.Cu) (net 39))
+  (segment (start 64.912501 67.167499) (end 64.399999 67.680001) (width 0.625) (layer F.Cu) (net 39))
+  (segment (start 77.327499 67.167499) (end 64.912501 67.167499) (width 0.625) (layer F.Cu) (net 39))
+  (segment (start 78.74 68.58) (end 77.327499 67.167499) (width 0.625) (layer F.Cu) (net 39))
+  (segment (start 131.180001 67.680001) (end 132.08 68.58) (width 0.625) (layer F.Cu) (net 39))
+  (segment (start 130.667499 67.167499) (end 131.180001 67.680001) (width 0.625) (layer F.Cu) (net 39))
+  (segment (start 118.252501 67.167499) (end 130.667499 67.167499) (width 0.625) (layer F.Cu) (net 39))
+  (segment (start 116.84 68.58) (end 118.252501 67.167499) (width 0.625) (layer F.Cu) (net 39))
+  (via (at 111 104) (size 0.8) (drill 0.4) (layers F.Cu B.Cu) (net 39))
+  (segment (start 106.68 114.3) (end 106.68 108.32) (width 0.625) (layer B.Cu) (net 39))
+  (segment (start 106.68 108.32) (end 111 104) (width 0.625) (layer B.Cu) (net 39))
+  (segment (start 116.84 98.16) (end 116.84 68.58) (width 0.625) (layer F.Cu) (net 39))
+  (segment (start 111 104) (end 116.84 98.16) (width 0.625) (layer F.Cu) (net 39))
+  (via (at 81 79) (size 0.8) (drill 0.4) (layers F.Cu B.Cu) (net 39))
+  (segment (start 116.84 68.58) (end 91.42 68.58) (width 0.625) (layer B.Cu) (net 39))
+  (segment (start 91.42 68.58) (end 81 79) (width 0.625) (layer B.Cu) (net 39))
+  (segment (start 78.74 76.74) (end 78.74 68.58) (width 0.625) (layer F.Cu) (net 39))
+  (segment (start 81 79) (end 78.74 76.74) (width 0.625) (layer F.Cu) (net 39))
   (segment (start 83.4009 151.9809) (end 83.82 151.9809) (width 0.25) (layer F.Cu) (net 40))
   (segment (start 78.74 147.32) (end 83.4009 151.9809) (width 0.25) (layer F.Cu) (net 40))
@@
   (segment (start 71.12 137.16) (end 71.12 139.7) (width 0.25) (layer F.Cu) (net 50))
   (segment (start 96.52 119.38) (end 96.52 121.92) (width 0.25) (layer F.Cu) (net 51))
+  (segment (start 96.52 137.16) (end 96.52 139.7) (width 0.25) (layer F.Cu) (net 51))
+  (via (at 95 127) (size 0.8) (drill 0.4) (layers F.Cu B.Cu) (net 51))
+  (segment (start 96.52 121.92) (end 96.52 125.48) (width 0.25) (layer F.Cu) (net 51))
+  (segment (start 96.52 125.48) (end 95 127) (width 0.25) (layer F.Cu) (net 51))
+  (segment (start 96.52 128.52) (end 96.52 137.16) (width 0.25) (layer B.Cu) (net 51))
+  (segment (start 95 127) (end 96.52 128.52) (width 0.25) (layer B.Cu) (net 51))
   (segment (start 88.9 137.16) (end 88.9 139.7) (width 0.25) (layer F.Cu) (net 52))
   (segment (start 91.44 137.16) (end 91.44 139.7) (width 0.25) (layer F.Cu) (net 53))
@@
   (segment (start 107.992501 118.152501) (end 107.992501 95.295066) (width 0.625) (layer F.Cu) (net 55))
   (segment (start 109.22 119.38) (end 107.992501 118.152501) (width 0.625) (layer F.Cu) (net 55))
+  (zone (net 1) (net_name GND) (layer F.Cu) (hatch edge 0.508)
+    (connect_pads (clearance 0.508))
+    (min_thickness 0.254)
+    (fill yes (arc_segments 16) (thermal_gap 0.508) (thermal_bridge_width 0.508))
+    (polygon
+      (pts
+        (xy 50 25) (xy 150 25) (xy 150 175) (xy 50 175)
+      )
+    )
+  )
+  (zone (net 1) (net_name GND) (layer B.Cu) (hatch edge 0.508)
+    (connect_pads (clearance 0.508))
+    (min_thickness 0.254)
+    (fill yes (arc_segments 16) (thermal_gap 0.508) (thermal_bridge_width 0.508))
+    (polygon
+      (pts
+        (xy 50 25) (xy 150 25) (xy 150 175) (xy 50 175)
+      )
+    )
+  )
 )
