File: pcb/v8/drumkid.sch (KiCad schematic (older format))
At the start: 57 parts, among them J1 DIN-5_180degree, J2 DIN-5_180degree, J3 Conn_01x15, J4 Conn_01x15, J9 AudioJack3_Ground_Switch, SW1 SW_Push, SW2 SW_Push, SW3 SW_Push, SW4 SW_Push, SW5 SW_Push, SW6 SW_Push, SW7 SW_SPDT, SW8 SW_SPDT, U1 6N138

Commit message: v8 layout looks decent
Parts:
- C1, C3: value CP -> 470uF; footprint Capacitor_THT:CP_Radial_D6.3mm_P2.50mm -> drumkidcustom:CP_Radial_D6.3mm_P2.50mm
- C2, C4: footprint Capacitor_THT:C_Disc_D3.4mm_W2.1mm_P2.50mm -> drumkidcustom:C_Disc_D3.4mm_W2.1mm_P2.50mm
- C5: renamed from C?; footprint (none) -> drumkidcustom:CP_Radial_D6.3mm_P2.50mm
- R12, R13: renamed from R?; footprint (none) -> drumkidcustom:R_Axial_DIN0207_L6.3mm_D2.5mm_P10.16mm_Horizontal
Changed lines of the file:
@@
 P 2950 1350
 F 0 "C1" H 3068 1396 50  0000 L CNN
-F 1 "CP" H 3068 1305 50  0000 L CNN
-F 2 "Capacitor_THT:CP_Radial_D6.3mm_P2.50mm" H 2988 1200 50  0001 C CNN
+F 1 "470uF" H 3068 1305 50  0000 L CNN
+F 2 "drumkidcustom:CP_Radial_D6.3mm_P2.50mm" H 2988 1200 50  0001 C CNN
 F 3 "~" H 2950 1350 50  0001 C CNN
 	1    2950 1350
@@
 F 0 "C2" H 3415 1396 50  0000 L CNN
 F 1 "C" H 3415 1305 50  0000 L CNN
-F 2 "Capacitor_THT:C_Disc_D3.4mm_W2.1mm_P2.50mm" H 3338 1200 50  0001 C CNN
+F 2 "drumkidcustom:C_Disc_D3.4mm_W2.1mm_P2.50mm" H 3338 1200 50  0001 C CNN
 F 3 "~" H 3300 1350 50  0001 C CNN
 	1    3300 1350
@@
 P 4800 5550
 F 0 "C3" H 4918 5596 50  0000 L CNN
-F 1 "CP" H 4918 5505 50  0000 L CNN
-F 2 "Capacitor_THT:CP_Radial_D6.3mm_P2.50mm" H 4838 5400 50  0001 C CNN
+F 1 "470uF" H 4918 5505 50  0000 L CNN
+F 2 "drumkidcustom:CP_Radial_D6.3mm_P2.50mm" H 4838 5400 50  0001 C CNN
 F 3 "~" H 4800 5550 50  0001 C CNN
 	1    4800 5550
@@
 F 0 "C4" H 5265 5596 50  0000 L CNN
 F 1 "C" H 5265 5505 50  0000 L CNN
-F 2 "Capacitor_THT:C_Disc_D3.4mm_W2.1mm_P2.50mm" H 5188 5400 50  0001 C CNN
+F 2 "drumkidcustom:C_Disc_D3.4mm_W2.1mm_P2.50mm" H 5188 5400 50  0001 C CNN
 F 3 "~" H 5150 5550 50  0001 C CNN
 	1    5150 5550
@@
 	2200 1000 2200 1450
 $Comp
-L Device:CP C?
+L Device:CP C5
 U 1 1 5EF27403
 P 8250 5300
-F 0 "C?" V 8505 5300 50  0000 C CNN
+F 0 "C5" V 8505 5300 50  0000 C CNN
 F 1 "22uF" V 8414 5300 50  0000 C CNN
-F 2 "" H 8288 5150 50  0001 C CNN
+F 2 "drumkidcustom:CP_Radial_D6.3mm_P2.50mm" H 8288 5150 50  0001 C CNN
 F 3 "~" H 8250 5300 50  0001 C CNN
 	1    8250 5300
@@
 $EndComp
 $Comp
-L Device:R R?
+L Device:R R13
 U 1 1 5EF29817
 P 9350 5500
-F 0 "R?" V 9450 5500 50  0000 C CNN
+F 0 "R13" V 9450 5500 50  0000 C CNN
 F 1 "1k" V 9550 5500 50  0000 C CNN
-F 2 "" V 9280 5500 50  0001 C CNN
+F 2 "drumkidcustom:R_Axial_DIN0207_L6.3mm_D2.5mm_P10.16mm_Horizontal" V 9280 5500 50  0001 C CNN
 F 3 "~" H 9350 5500 50  0001 C CNN
 	1    9350 5500
@@
 $EndComp
 $Comp
-L Device:R R?
+L Device:R R12
 U 1 1 5EF282B1
 P 9350 5300
-F 0 "R?" V 9143 5300 50  0000 C CNN
+F 0 "R12" V 9143 5300 50  0000 C CNN
 F 1 "1k" V 9234 5300 50  0000 C CNN
-F 2 "" V 9280 5300 50  0001 C CNN
+F 2 "drumkidcustom:R_Axial_DIN0207_L6.3mm_D2.5mm_P10.16mm_Horizontal" V 9280 5300 50  0001 C CNN
 F 3 "~" H 9350 5300 50  0001 C CNN
 	1    9350 5300
