File: pcb/v8/drumkid.kicad_pcb (KiCad board)
At the start: 2 copper layers, 90 x 140 mm, 54 parts, among them J1 DIN-5_180degree, J2 DIN-5_180degree, J3 Conn_01x15, J4 Conn_01x15, J9 AudioJack3_Ground_Switch, SW1 SW_Push, SW2 SW_Push, SW3 SW_Push, SW4 SW_Push, SW5 SW_Push, SW6 SW_Push, SW7 SW_SPDT, SW8 SW_SPDT, U1 6N138

Commit message: v8 layout looks decent
Parts:
- added C5: 22uF, drumkidcustom:CP_Radial_D6.3mm_P2.50mm, F.Cu at (110.5, 138.4)
- added R12: 1k, drumkidcustom:R_Axial_DIN0207_L6.3mm_D2.5mm_P10.16mm_Horizontal, F.Cu at (118.1, 143.5)
- added R13: 1k, drumkidcustom:R_Axial_DIN0207_L6.3mm_D2.5mm_P10.16mm_Horizontal, F.Cu at (120.7, 143.5)
- C1, C3: value CP -> 470uF
Connections:
- J9 pad T: Net-(J9-PadR) -> Net-(J9-PadT)
- RV5 pad 2: Net-(J9-PadR) -> Net-(C5-Pad1)
Routing:
- net Net-(J9-PadT): track 0.00 -> 145.5 mm
- net Net-(C5-Pad1): track 0.00 -> 127.9 mm
- net Net-(J9-PadR): track 27.4 -> 152.5 mm
- net Net-(C5-Pad2): track 0.00 -> 9.76 mm
- net /DIGITAL_0: track 44.2 -> 47.8 mm
Other:
- board text added: "DrumKid v08 by Matt Bradshaw mattbradshawdesign.com github.com/mattybrad/drumkid"
- board text removed: "DrumKid v07 by Matt Bradshaw mattbradshawdesign.com github.com/mattybrad/drumkid"

Commit message: v8 gerbers done
Routing:
- net Net-(D3-Pad2): track 112.5 -> 100.6 mm
- net Net-(D2-Pad2): track 102.1 -> 95.4 mm
- net Net-(C5-Pad1): track 127.9 -> 123.9 mm
- net Net-(D1-Pad2): track 89.8 -> 92.1 mm
- net Net-(J9-PadT): track 145.5 -> 145.0 mm
