File: pcb/v10smt/drumkid.sch (KiCad schematic (older format))
At the start: 63 parts, among them J1 DIN-5_180degree, J2 DIN-5_180degree, J3 Conn_01x15, J4 Conn_01x15, J9 AudioJack3_Ground_Switch, SW1 SW_Push, SW2 SW_Push, SW3 SW_Push, SW4 SW_Push, SW5 SW_Push, SW6 SW_Push, SW7 SW_SPDT, SW8 SW_SPDT, U1 6N138

Commit message: another new PCB revision, hopefully the last one for a while...
Parts:
- removed C?: 100nF, symbol Device:C
- removed D8: 1N5817, Diode_THT:D_DO-41_SOD81_P10.16mm_Horizontal, symbol Diode:1N5817
- removed J? (x2): Conn_01x15, Connector_PinSocket_2.54mm:PinSocket_1x15_P2.54mm_Vertical, symbol Connector_Generic:Conn_01x15
- removed J? (x4): Conn_01x10, symbol Connector_Generic:Conn_01x10
- removed R?: 270, drumkidcustom:R_Axial_DIN0207_L6.3mm_D2.5mm_P10.16mm_Horizontal, symbol Device:R
- added C2, C4: C, drumkidcustom:C_Disc_D3.4mm_W2.1mm_P2.50mm, symbol Device:C
- added D8: 1N4001, Diode_SMD:D_SOD-123, symbol Diode:1N4001
- BT1: footprint Connector_Wire:SolderWirePad_1x02_P5.08mm_Drill1.5mm -> Connector_Wire:SolderWire-0.5sqmm_1x02_P4.8mm_D0.9mm_OD2.3mm
- C1, C3, C5: footprint drumkidcustom:CP_Radial_D6.3mm_P2.50mm -> Capacitor_SMD:CP_Elec_8x10
- D7: footprint Diode_THT:D_DO-35_SOD27_P7.62mm_Horizontal -> Diode_SMD:D_SOD-323
- R1, R2, R3, R4, R5, R6: value R_LED -> 680; footprint drumkidcustom:R_Axial_DIN0207_L6.3mm_D2.5mm_P10.16mm_Horizontal -> Resistor_SMD:R_1206_3216Metric
- R10, R11, R12, R13, R7, R8, R9: footprint drumkidcustom:R_Axial_DIN0207_L6.3mm_D2.5mm_P10.16mm_Horizontal -> Resistor_SMD:R_1206_3216Metric
- U1: footprint Package_DIP:DIP-8_W7.62mm_Socket -> Package_DIP:PowerIntegrations_SMD-8
Connections:
- wire segments 132 -> 107
Other:
- moved on the sheet: C5, H1, H10, H2, H3, H4, H5, H6, H7, H8, H9, J9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
