File: pcb/v9/drumkid.kicad_pcb (KiCad board)
At the start: 2 copper layers, 90 x 140 mm, 57 parts, among them J1 DIN-5_180degree, J2 DIN-5_180degree, J3 Conn_01x15, J4 Conn_01x15, J9 AudioJack3_Ground_Switch, SW1 SW_Push, SW2 SW_Push, SW3 SW_Push, SW4 SW_Push, SW5 SW_Push, SW6 SW_Push, SW7 SW_SPDT, SW8 SW_SPDT, U1 6N138

Commit message: another new PCB revision, hopefully the last one for a while...
Parts:
- A1, J1, J2, J3, J4, SW8: moved to F.Cu
- BT1: footprint Connector_Wire:SolderWire-0.5sqmm_1x02_P4.8mm_D0.9mm_OD2.3mm -> Connector_Wire:SolderWirePad_1x02_P5.08mm_Drill1.5mm; moved to F.Cu
- C1, C3: footprint Capacitor_SMD:CP_Elec_8x10 -> Capacitor_THT:CP_Radial_D6.3mm_P2.50mm; moved to F.Cu
- C2, C4: footprint drumkidcustom:C_Disc_D3.4mm_W2.1mm_P2.50mm -> Capacitor_THT:C_Disc_D3.4mm_W2.1mm_P2.50mm; moved to F.Cu
- C5: footprint Capacitor_SMD:CP_Elec_8x10 -> drumkidcustom:CP_Radial_D6.3mm_P2.50mm; moved to F.Cu
- D1, D2, D3, D4, D5, D6, H10, H9, J9, RV1, RV2, RV3, RV4, RV5, SW1, SW2, SW3, SW4, SW5, SW6, SW7: moved to B.Cu
- D7: footprint Diode_SMD:D_SOD-323 -> Diode_THT:D_DO-35_SOD27_P7.62mm_Horizontal; moved to F.Cu
- D8: value 1N4001 -> 1N5817; footprint Diode_SMD:D_SOD-123 -> Diode_THT:D_DO-41_SOD81_P10.16mm_Horizontal; moved to F.Cu
- R1, R10, R11, R12, R13, R2, R3, R4, R5, R6, R7, R8, R9: footprint Resistor_SMD:R_1206_3216Metric -> drumkidcustom:R_Axial_DIN0207_L6.3mm_D2.5mm_P10.16mm_Horizontal; moved to F.Cu
- U1: footprint Package_DIP:PowerIntegrations_SMD-8 -> Package_DIP:DIP-8_W7.62mm_Socket; moved to F.Cu
- moved H7 114.0 mm to (100.0, 50.0)
- moved R12 111.2 mm to (118.1, 143.5), turned to 90 degrees
- moved H2 106.3 mm to (60.0, 105.0)
- moved R13 104.6 mm to (120.7, 143.5), turned to 90 degrees
- moved C5 97.7 mm to (110.5, 138.4)
- moved D8 97.4 mm to (109.2, 129.5), turned to 90 degrees
- moved H8 85.4 mm to (100.0, 80.0)
- moved H3 80.6 mm to (70.0, 160.0)
- moved H4 80.6 mm to (130.0, 160.0)
- moved H5 80.0 mm to (140.0, 105.0)
- moved SW1 78.2 mm to (134.6, 81.3), turned to 270 degrees
- moved SW6 75.7 mm to (61.0, 81.3), turned to 270 degrees
- moved H6 70.0 mm to (140.0, 35.0)
- moved J3 69.0 mm to (66.0, 139.7)
- moved J4 69.0 mm to (66.0, 119.4)
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Routing:
- net VCC: track 0.00 -> 256.7 mm, vias 0 -> 2
- net /ANALOG_1: track 0.00 -> 176.5 mm
- net /ANALOG_0: track 0.00 -> 168.5 mm
- net Net-(J9-PadR): track 0.00 -> 152.5 mm
- net Net-(J9-PadT): track 0.00 -> 145.0 mm
- net Net-(C5-Pad1): track 0.00 -> 123.9 mm
- net Net-(D8-Pad2): track 0.00 -> 101.5 mm
- net Net-(D3-Pad2): track 0.00 -> 100.6 mm
- net /DIGITAL_9: track 0.00 -> 96.4 mm
- net Net-(D2-Pad2): track 0.00 -> 95.4 mm
- net Net-(D1-Pad2): track 0.00 -> 92.1 mm
- net Net-(BT1-Pad1): track 0.00 -> 89.3 mm
- net /DIGITAL_4: track 0.00 -> 85.3 mm
- net /ANALOG_3: track 0.00 -> 83.5 mm
- net /DIGITAL_5: track 0.00 -> 75.7 mm, vias 0 -> 1
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- added copper zone on B.Cu, net GND
- added copper zone on F.Cu, net GND
Other:
- board text added: "(change bank)"
- board text added: "(load)"
- board text added: "(save)"
- board text added: "+"
- board text added: "+ -"
- board text added: "0"
- board text added: "1"
- board text added: "1N4148"
- board text added: "1N5817"
- board text added: "6N138"
- board text added: "Arduino Nano 3"
- board text added: "DrumKid v08 by Matt Bradshaw mattbradshawdesign.com github.com/mattybrad/drumkid"
- board text added: "JLCJLCJLCJLC"
- board text added: "Serial number"
- board text added: "USB port this end"
- board text added: "a"
- board text added: "a b c d"
- board text added: "aleatoric drum machine"
- board text added: "arduino"
- board text added: "b"
- board text added: "c"
- board text added: "chance pitch drone beat"
- board text added: "d"
- board text added: "drumkid"
- board text added: "midi"
- board text added: "midi in"
- board text added: "midi out"
- board text added: "midpoint drop note tempo"
- board text added: "range crop tuning swing"
- board text added: "start/stop"
- board text added: "tap tempo"
- board text added: "zoom crush modulate beats/bar"

Commit message: making space for new bits
Parts:
- removed C4: C, Capacitor_THT:C_Disc_D3.4mm_W2.1mm_P2.50mm
- added J10: Conn_01x15, Connector_PinSocket_2.54mm:PinSocket_1x15_P2.54mm_Vertical, F.Cu at (66.0, 134.6)
- added J11: Conn_01x15, Connector_PinSocket_2.54mm:PinSocket_1x15_P2.54mm_Vertical, F.Cu at (66.0, 124.5)
- added J5: Conn_01x10, Connector_PinSocket_2.54mm:PinSocket_1x10_P2.54mm_Vertical, F.Cu at (109.2, 147.3)
- added J6: Conn_01x10, Connector_PinSocket_2.54mm:PinSocket_1x10_P2.54mm_Vertical, F.Cu at (109.2, 144.8)
- added J7: Conn_01x10, Connector_PinSocket_2.54mm:PinSocket_1x10_P2.54mm_Vertical, F.Cu at (109.2, 106.7)
- added J8: Conn_01x10, Connector_PinSocket_2.54mm:PinSocket_1x10_P2.54mm_Vertical, F.Cu at (109.2, 104.1)
- added R14: 270, drumkidcustom:R_Axial_DIN0207_L6.3mm_D2.5mm_P10.16mm_Horizontal, F.Cu at (63.5, 114.3)
- C1, C3: footprint Capacitor_THT:CP_Radial_D6.3mm_P2.50mm -> drumkidcustom:CP_Radial_D6.3mm_P2.50mm
- C2: value C -> 100nF; footprint Capacitor_THT:C_Disc_D3.4mm_W2.1mm_P2.50mm -> Capacitor_THT:C_Disc_D3.0mm_W1.6mm_P2.50mm
- R1, R2, R3, R4, R5, R6: value 680 -> R_LED
- moved C2 41.6 mm to (76.2, 114.3), turned to 0 degrees
- moved R7 18.5 mm to (124.5, 152.4)
- moved SW8 11.7 mm to (132.1, 135.9)
- moved R8 7.62 mm to (137.2, 121.9)
- moved R9 7.62 mm to (134.6, 111.8)
- moved U1 7.62 mm to (121.9, 111.8)
- moved R12 5.39 mm to (121.9, 139.7)
- moved R13 5.39 mm to (124.5, 139.7)
- moved C5 3.59 mm to (113.0, 135.9)
- moved J1 1.68 mm to (110.0, 158.0)
- moved J2 1.29 mm to (90.0, 158.0)
Connections:
- C2 pad 1: VCC -> Net-(C2-Pad1)
- RV5 pad 1: /DIGITAL_9 -> Net-(C2-Pad1)
Routing:
- net VCC: track 256.7 -> 0.00 mm, vias 2 -> 0
- net /ANALOG_1: track 176.5 -> 0.00 mm
- net /ANALOG_0: track 168.5 -> 0.00 mm
- net Net-(J9-PadR): track 152.5 -> 0.00 mm
- net Net-(J9-PadT): track 145.0 -> 0.00 mm
- net Net-(C5-Pad1): track 123.9 -> 0.00 mm
- net Net-(D8-Pad2): track 101.5 -> 0.00 mm
- net Net-(D3-Pad2): track 100.6 -> 0.00 mm
- net /DIGITAL_9: track 96.4 -> 0.00 mm
- net Net-(D2-Pad2): track 95.4 -> 0.00 mm
- net Net-(D1-Pad2): track 92.1 -> 0.00 mm
- net Net-(BT1-Pad1): track 89.3 -> 0.00 mm
- net /DIGITAL_4: track 85.3 -> 0.00 mm
- net /ANALOG_3: track 83.5 -> 0.00 mm
- net /DIGITAL_5: track 75.7 -> 0.00 mm, vias 1 -> 0
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- removed copper zone on B.Cu, net GND
- removed copper zone on F.Cu, net GND

Commit message: may have squeezed too many things onto the PCB...
Parts:
- added J12: Conn_01x05, Connector_PinSocket_2.54mm:PinSocket_1x05_P2.54mm_Vertical, F.Cu at (73.7, 144.8)
- added J13: AudioJack3_Ground_Switch, drumkidcustom:Tayda_3.5mm_stereo_TRS_jack_A-853, F.Cu at (65.1, 149.9)
- added J14: Conn_01x05, Connector_PinSocket_2.54mm:PinSocket_1x05_P2.54mm_Vertical, F.Cu at (129.5, 121.9)
- added J15: AudioJack3_Ground_Switch, drumkidcustom:Tayda_3.5mm_stereo_TRS_jack_A-853, F.Cu at (138.0, 116.8)
- J10, J11: footprint Connector_PinSocket_2.54mm:PinSocket_1x15_P2.54mm_Vertical -> Connector_PinHeader_2.54mm:PinHeader_1x15_P2.54mm_Vertical
- J6, J7: footprint Connector_PinSocket_2.54mm:PinSocket_1x10_P2.54mm_Vertical -> Connector_PinHeader_2.54mm:PinHeader_1x10_P2.54mm_Vertical
- moved R8 12.7 mm to (124.5, 121.9)
- moved R9 12.7 mm to (121.9, 111.8)
- moved U1 10.2 mm to (111.8, 111.8)
- moved D8 5.08 mm to (109.2, 134.6)
- moved D7 5.08 mm to (116.8, 124.5)
- moved C5 1.27 mm to (113.0, 137.2)
Other:
- board text added: "DrumKid v9 by Matt Bradshaw mattbradshawdesign.com github.com/mattybrad/drumkid"
- board text removed: "DrumKid v08 by Matt Bradshaw mattbradshawdesign.com github.com/mattybrad/drumkid"

Commit message: routing...
Routing:
- net Net-(C2-Pad1): track 0.00 -> 143.0 mm
- net Net-(J9-PadR): track 0.00 -> 120.1 mm
- net Net-(J9-PadT): track 0.00 -> 111.3 mm
- net Net-(D8-Pad2): track 0.00 -> 101.3 mm
- net Net-(C5-Pad1): track 0.00 -> 95.6 mm
- net Net-(BT1-Pad1): track 0.00 -> 72.0 mm
- net VCC: track 0.00 -> 42.8 mm
- net Net-(J2-Pad4): track 0.00 -> 19.5 mm
- net /DIGITAL_8: track 0.00 -> 17.6 mm
- net /DIGITAL_7: track 0.00 -> 17.6 mm
- net /DIGITAL_6: track 0.00 -> 17.6 mm
- net /DIGITAL_5: track 0.00 -> 17.6 mm
- net /DIGITAL_4: track 0.00 -> 17.6 mm
- net /DIGITAL_10: track 0.00 -> 17.6 mm
- net GND: track 0.00 -> 16.3 mm
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
Commit message: more routing, going well...
Routing:
- net VCC: track 42.8 -> 291.6 mm
- net /ANALOG_1: track 5.08 -> 182.2 mm
- net /ANALOG_0: track 5.08 -> 172.6 mm
- net /ANALOG_2: track 5.08 -> 109.7 mm
- net Net-(D3-Pad2): track 0.00 -> 95.2 mm
- net /ANALOG_3: track 5.08 -> 94.0 mm
- net Net-(D6-Pad2): track 0.00 -> 77.4 mm
- net /DIGITAL_11: track 5.08 -> 76.1 mm
- net Net-(D1-Pad2): track 0.00 -> 70.4 mm
- net /DIGITAL_4: track 17.6 -> 78.9 mm
- net Net-(D2-Pad2): track 0.00 -> 61.3 mm
- net Net-(D5-Pad2): track 0.00 -> 56.1 mm
- net /DIGITAL_5: track 17.6 -> 73.7 mm
- net Net-(D4-Pad2): track 0.00 -> 55.2 mm
- net Net-(D7-Pad1): track 0.00 -> 47.5 mm
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