File: pcb/v9/drumkid.kicad_pcb (KiCad board)
At the start: 2 copper layers, 90 x 140 mm, 67 parts, among them J1 DIN-5_180degree, J10 Conn_01x15, J11 Conn_01x15, J12 Conn_01x05, J13 AudioJack3_Ground_Switch, J14 Conn_01x05, J15 AudioJack3_Ground_Switch, J2 DIN-5_180degree, J3 Conn_01x15, J4 Conn_01x15, J5 Conn_01x10, J6 Conn_01x10, J7 Conn_01x10, J8 Conn_01x10, J9 AudioJack3_Ground_Switch, SW1 SW_Push, SW2 SW_Push, SW3 SW_Push, SW4 SW_Push, SW5 SW_Push, SW6 SW_Push, SW7 SW_SPDT, SW8 SW_SPDT, U1 6N138

Commit message: omg that's the best routing i've ever done
Routing:
- net Net-(D7-Pad2): track 18.0 -> 69.5 mm
- net /DIGITAL_2: track 5.08 -> 19.9 mm
- net /DIGITAL_3: track 5.08 -> 19.9 mm
- net /RESET: track 10.2 -> 20.3 mm
- net Net-(D7-Pad1): track 47.5 -> 48.2 mm
- added copper zone on B.Cu, net GND
- added copper zone on F.Cu, net GND

Commit message: minor silkscreen edits
Routing:
- net GND: vias 0 -> 13
Other:
- board text added: "R RN S TN T"
- board text added: "T TN S RN R"
Changed lines of the file:
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@@
   (general
     (thickness 1.6)
-    (drawings 78)
-    (tracks 437)
+    (drawings 80)
+    (tracks 450)
     (zones 0)
     (modules 67)
@@
     (tags connector)
     (attr virtual)
-    (fp_text reference BT1 (at 2.88 2.32) (layer F.SilkS)
+    (fp_text reference BT1 (at 8.89 -0.635) (layer F.SilkS)
       (effects (font (size 1 1) (thickness 0.15)))
     )
-    (fp_text value Battery (at 2.54 3.81) (layer F.Fab)
+    (fp_text value Battery (at 2.54 3.81) (layer F.SilkS)
       (effects (font (size 1 1) (thickness 0.15)))
     )
@@
     (descr "CP, Radial series, Radial, pin pitch=2.50mm, , diameter=6.3mm, Electrolytic Capacitor")
     (tags "CP Radial series Radial pin pitch 2.50mm  diameter 6.3mm Electrolytic Capacitor")
-    (fp_text reference C1 (at 1.25 -4.4) (layer F.SilkS)
+    (fp_text reference C1 (at 5.08 -1.905) (layer F.SilkS)
       (effects (font (size 1 1) (thickness 0.15)))
     )
@@
       (effects (font (size 1 1) (thickness 0.15)))
     )
-    (fp_text value 100nF (at 1.25 2.05) (layer F.Fab)
+    (fp_text value 100nF (at 1.25 2.05) (layer F.SilkS)
       (effects (font (size 1 1) (thickness 0.15)))
     )
@@
     )
   )
+  (gr_text "T\nTN\nS\nRN\nR" (at 128.27 116.84) (layer F.SilkS)
+    (effects (font (size 1.5 1) (thickness 0.25)) (justify right))
+  )
+  (gr_text "R\nRN\nS\nTN\nT" (at 74.93 149.86) (layer F.SilkS)
+    (effects (font (size 1.5 1) (thickness 0.25)) (justify left))
+  )
   (gr_text "DrumKid v9\nby Matt Bradshaw\nmattbradshawdesign.com\ngithub.com/mattybrad/drumkid" (at 93.5 98) (layer F.SilkS)
     (effects (font (size 1.2 1.2) (thickness 0.2)) (justify left))
@@
     (effects (font (size 1.2 1.2) (thickness 0.3)) (justify mirror))
   )
-  (gr_text JLCJLCJLCJLC (at 88.9 132.08) (layer F.SilkS)
+  (gr_text JLCJLCJLCJLC (at 99.695 55.88) (layer F.SilkS)
     (effects (font (size 1 1) (thickness 0.15)))
   )
-  (gr_text 6N138 (at 109.22 116.84 90) (layer F.SilkS)
+  (gr_text 6N138 (at 115.57 121.92) (layer F.SilkS)
     (effects (font (size 1 1) (thickness 0.2)))
   )
@@
   (segment (start 124.46 123.05137) (end 124.278869 123.232501) (width 0.625) (layer F.Cu) (net 1))
   (segment (start 124.46 121.92) (end 124.46 123.05137) (width 0.625) (layer F.Cu) (net 1))
+  (via (at 91.44 129.54) (size 0.8) (drill 0.4) (layers F.Cu B.Cu) (net 1))
+  (via (at 81.28 129.54) (size 0.8) (drill 0.4) (layers F.Cu B.Cu) (net 1))
+  (via (at 124.46 116.84) (size 0.8) (drill 0.4) (layers F.Cu B.Cu) (net 1))
+  (via (at 93.98 106.68) (size 0.8) (drill 0.4) (layers F.Cu B.Cu) (net 1))
+  (via (at 60.96 116.84) (size 0.8) (drill 0.4) (layers F.Cu B.Cu) (net 1))
+  (via (at 101.6 149.86) (size 0.8) (drill 0.4) (layers F.Cu B.Cu) (net 1))
+  (via (at 91.44 160.02) (size 0.8) (drill 0.4) (layers F.Cu B.Cu) (net 1))
+  (via (at 109.22 160.02) (size 0.8) (drill 0.4) (layers F.Cu B.Cu) (net 1))
+  (via (at 63.5 144.78) (size 0.8) (drill 0.4) (layers F.Cu B.Cu) (net 1))
+  (via (at 134.62 109.22) (size 0.8) (drill 0.4) (layers F.Cu B.Cu) (net 1))
+  (via (at 66.04 109.22) (size 0.8) (drill 0.4) (layers F.Cu B.Cu) (net 1))
+  (via (at 58.42 129.54) (size 0.8) (drill 0.4) (layers F.Cu B.Cu) (net 1))
+  (via (at 139.7 147.32) (size 0.8) (drill 0.4) (layers F.Cu B.Cu) (net 1))
   (segment (start 81.28 139.7) (end 81.28 134.62) (width 0.25) (layer F.Cu) (net 4))
   (segment (start 58.074999 73.075999) (end 58.074999 125.067499) (width 0.25) (layer B.Cu) (net 4))
