File: pcb/v10/drumkid.kicad_pcb (KiCad board)
At the start: 2 copper layers, 90 x 140 mm, 67 parts, among them J1 DIN-5_180degree, J10 Conn_01x15, J11 Conn_01x15, J12 Conn_01x05, J13 AudioJack3_Ground_Switch, J14 Conn_01x05, J15 AudioJack3_Ground_Switch, J2 DIN-5_180degree, J3 Conn_01x15, J4 Conn_01x15, J5 Conn_01x10, J6 Conn_01x10, J7 Conn_01x10, J8 Conn_01x10, J9 AudioJack3_Ground_Switch, SW1 SW_Push, SW2 SW_Push, SW3 SW_Push, SW4 SW_Push, SW5 SW_Push, SW6 SW_Push, SW7 SW_SPDT, SW8 SW_SPDT, U1 6N138

Commit message: v10 pcb
Parts:
- R12, R13: value 1k -> 220

Commit message: nice new logo
Parts:
- added U2: LOGO, drumkidcustom:drumkid_logo, B.Cu at (100.4, 59.1)
Other:
- board text added: "DrumKid v10 by Matt Bradshaw mattbradshawdesign.com github.com/mattybrad/drumkid"
- board text removed: "DrumKid v9 by Matt Bradshaw mattbradshawdesign.com github.com/mattybrad/drumkid"
- board text removed: "drumkid"

Commit message: v10 pcb done
Parts:
- added U3: drumkid_logo, drumkidcustom:drumkid_logo, F.Cu at (100.3, 57.0)
- R1, R2, R3, R4, R5, R6: value R_LED -> 680*
- U2: value LOGO -> drumkid_logo
- moved U2 0.66 mm to (100.5, 59.8)
Other:
- board text added: "LEDs mounted on other side"
- board text added: "MIDI sockets mounted this side"
- board text added: "This is the underside of the PCB, which will not be seen. Solder in this order: resistors, diodes, IC socket, MIDI switch, 15-pin headers, capacitors, audio socket, power switch, buttons, LEDs, potentiometers, MIDI sockets, battery leads"
- board text added: "buttons mounted on other side"
- board text added: "don't solder the nano to the board! solder the two 15-pins headers, using the middle rows."
- board text added: "potentiometers mounted on other side"
- board text added: "power switch, audio output and volume pot mounted on other side"
- board text added: "the outlined areas are reserved for user modifications, and should not be populated initially"
