File: pcb/v10/drumkid.sch (KiCad schematic (older format))
At the start: 67 parts, among them J1 DIN-5_180degree, J10 Conn_01x15, J11 Conn_01x15, J12 Conn_01x05, J13 AudioJack3_Ground_Switch, J14 Conn_01x05, J15 AudioJack3_Ground_Switch, J2 DIN-5_180degree, J3 Conn_01x15, J4 Conn_01x15, J5 Conn_01x10, J6 Conn_01x10, J7 Conn_01x10, J8 Conn_01x10, J9 AudioJack3_Ground_Switch, SW1 SW_Push, SW2 SW_Push, SW3 SW_Push, SW4 SW_Push, SW5 SW_Push, SW6 SW_Push, SW7 SW_SPDT, SW8 SW_SPDT, U1 6N138

Commit message: v10 pcb
Parts:
- R12, R13: value 1k -> 220
Changed lines of the file:
@@
 P 9750 5500
 F 0 "R13" V 9850 5500 50  0000 C CNN
-F 1 "1k" V 9950 5500 50  0000 C CNN
+F 1 "220" V 9950 5500 50  0000 C CNN
 F 2 "drumkidcustom:R_Axial_DIN0207_L6.3mm_D2.5mm_P10.16mm_Horizontal" V 9680 5500 50  0001 C CNN
 F 3 "~" H 9750 5500 50  0001 C CNN
@@
 P 9750 5300
 F 0 "R12" V 9543 5300 50  0000 C CNN
-F 1 "1k" V 9634 5300 50  0000 C CNN
+F 1 "220" V 9634 5300 50  0000 C CNN
 F 2 "drumkidcustom:R_Axial_DIN0207_L6.3mm_D2.5mm_P10.16mm_Horizontal" V 9680 5300 50  0001 C CNN
 F 3 "~" H 9750 5300 50  0001 C CNN

Commit message: nice new logo
Parts:
- added U2: drumkid_logo, drumkidcustom:drumkid_logo, symbol drumkidcustom:drumkid_logo
Changed lines of the file:
@@
 Wire Wire Line
 	4350 1000 4150 1000
+$Comp
+L drumkidcustom:drumkid_logo U2
+U 1 1 5FA091CC
+P 3250 4450
+F 0 "U2" H 3275 4496 50  0000 L CNN
+F 1 "drumkid_logo" H 3275 4405 50  0000 L CNN
+F 2 "drumkidcustom:drumkid_logo" H 3250 4450 50  0001 C CNN
+F 3 "" H 3250 4450 50  0001 C CNN
+	1    3250 4450
+	1    0    0    -1
+$EndComp
 $EndSCHEMATC

Commit message: v10 pcb done
Parts:
- added U3: drumkid_logo, drumkidcustom:drumkid_logo, symbol drumkidcustom:drumkid_logo
- R1, R2, R3, R4, R5, R6: value R_LED -> 680*
Changed lines of the file:
@@
 P 5450 1650
 F 0 "R1" V 5243 1650 50  0000 C CNN
-F 1 "R_LED" V 5334 1650 50  0000 C CNN
+F 1 "680*" V 5334 1650 50  0000 C CNN
 F 2 "drumkidcustom:R_Axial_DIN0207_L6.3mm_D2.5mm_P10.16mm_Horizontal" V 5380 1650 50  0001 C CNN
 F 3 "~" H 5450 1650 50  0001 C CNN
@@
 P 5450 2050
 F 0 "R2" V 5243 2050 50  0000 C CNN
-F 1 "R_LED" V 5334 2050 50  0000 C CNN
+F 1 "680*" V 5334 2050 50  0000 C CNN
 F 2 "drumkidcustom:R_Axial_DIN0207_L6.3mm_D2.5mm_P10.16mm_Horizontal" V 5380 2050 50  0001 C CNN
 F 3 "~" H 5450 2050 50  0001 C CNN
@@
 P 5450 2450
 F 0 "R3" V 5243 2450 50  0000 C CNN
-F 1 "R_LED" V 5334 2450 50  0000 C CNN
+F 1 "680*" V 5334 2450 50  0000 C CNN
 F 2 "drumkidcustom:R_Axial_DIN0207_L6.3mm_D2.5mm_P10.16mm_Horizontal" V 5380 2450 50  0001 C CNN
 F 3 "~" H 5450 2450 50  0001 C CNN
@@
 P 5450 3250
 F 0 "R5" V 5243 3250 50  0000 C CNN
-F 1 "R_LED" V 5334 3250 50  0000 C CNN
+F 1 "680*" V 5334 3250 50  0000 C CNN
 F 2 "drumkidcustom:R_Axial_DIN0207_L6.3mm_D2.5mm_P10.16mm_Horizontal" V 5380 3250 50  0001 C CNN
 F 3 "~" H 5450 3250 50  0001 C CNN
@@
 P 5450 3650
 F 0 "R6" V 5243 3650 50  0000 C CNN
-F 1 "R_LED" V 5334 3650 50  0000 C CNN
+F 1 "680*" V 5334 3650 50  0000 C CNN
 F 2 "drumkidcustom:R_Axial_DIN0207_L6.3mm_D2.5mm_P10.16mm_Horizontal" V 5380 3650 50  0001 C CNN
 F 3 "~" H 5450 3650 50  0001 C CNN
@@
 P 5450 2850
 F 0 "R4" V 5243 2850 50  0000 C CNN
-F 1 "R_LED" V 5334 2850 50  0000 C CNN
+F 1 "680*" V 5334 2850 50  0000 C CNN
 F 2 "drumkidcustom:R_Axial_DIN0207_L6.3mm_D2.5mm_P10.16mm_Horizontal" V 5380 2850 50  0001 C CNN
 F 3 "~" H 5450 2850 50  0001 C CNN
@@
 	1    0    0    -1
 $EndComp
+$Comp
+L drumkidcustom:drumkid_logo U3
+U 1 1 5FA312B5
+P 3900 4450
+F 0 "U3" H 3925 4496 50  0000 L CNN
+F 1 "drumkid_logo" H 3925 4405 50  0000 L CNN
+F 2 "drumkidcustom:drumkid_logo" H 3900 4450 50  0001 C CNN
+F 3 "" H 3900 4450 50  0001 C CNN
+	1    3900 4450
+	1    0    0    -1
+$EndComp
