File: pcb/v11/drumkid.kicad_pcb (KiCad board)
At the start: 2 copper layers, 90 x 140 mm, 69 parts, among them J1 DIN-5_180degree, J10 Conn_01x15, J11 Conn_01x15, J12 Conn_01x05, J13 AudioJack3_Ground_Switch, J14 Conn_01x05, J15 AudioJack3_Ground_Switch, J2 DIN-5_180degree, J3 Conn_01x15, J4 Conn_01x15, J5 Conn_01x10, J6 Conn_01x10, J7 Conn_01x10, J8 Conn_01x10, J9 AudioJack3_Ground_Switch, SW1 SW_Push, SW2 SW_Push, SW3 SW_Push, SW4 SW_Push, SW5 SW_Push, SW6 SW_Push, SW7 SW_SPDT, SW8 SW_SPDT, U1 6N138, U2 drumkid_logo, U3 drumkid_logo

Commit message: little manual update and new PCB in progress
Parts:
- removed U3: drumkid_logo, drumkidcustom:drumkid_logo
- C1, C3: footprint drumkidcustom:CP_Radial_D6.3mm_P2.50mm -> Capacitor_SMD:CP_Elec_6.3x7.7
- C2: footprint Capacitor_THT:C_Disc_D3.0mm_W1.6mm_P2.50mm -> Capacitor_SMD:C_0402_1005Metric
- C5: footprint drumkidcustom:CP_Radial_D6.3mm_P2.50mm -> Capacitor_SMD:C_0603_1608Metric
- D7: footprint Diode_THT:D_DO-35_SOD27_P7.62mm_Horizontal -> Diode_SMD:D_SOD-123
- D8: footprint Diode_THT:D_DO-41_SOD81_P10.16mm_Horizontal -> Diode_SMD:D_SOD-123
- R1, R10, R11, R12, R13, R14, R2, R3, R4, R5, R6, R7, R8, R9: footprint drumkidcustom:R_Axial_DIN0207_L6.3mm_D2.5mm_P10.16mm_Horizontal -> Resistor_SMD:R_0805_2012Metric
- U1: footprint Package_DIP:DIP-8_W7.62mm_Socket -> Package_DIP:PowerIntegrations_SMD-8
- moved R4 46.9 mm to (97.9, 58.1)
- moved R5 46.9 mm to (95.4, 58.1)
- moved R6 46.9 mm to (92.8, 58.1)
- moved R1 46.0 mm to (105.7, 58.1)
- moved R2 46.0 mm to (103.1, 58.1)
- moved R3 46.0 mm to (100.6, 58.1)
- moved R9 2.75 mm to (122.2, 114.5)
- moved R7 2.45 mm to (122.8, 154.2)
- moved C2 1.28 mm to (76.9, 113.2)
- moved C3 0.30 mm to (94.0, 114.0)
Routing:
- net VCC: track 291.6 -> 0.00 mm
- net /ANALOG_1: track 182.2 -> 0.00 mm
- net /ANALOG_0: track 172.6 -> 0.00 mm
- net Net-(C2-Pad1): track 143.0 -> 0.00 mm
- net Net-(J9-PadR): track 120.1 -> 0.00 mm
- net Net-(J9-PadT): track 111.3 -> 0.00 mm
- net /ANALOG_2: track 109.7 -> 0.00 mm
- net Net-(D8-Pad2): track 101.3 -> 0.00 mm
- net Net-(C5-Pad1): track 95.6 -> 0.00 mm
- net Net-(D3-Pad2): track 95.2 -> 0.00 mm
- net /ANALOG_3: track 94.0 -> 0.00 mm
- net /DIGITAL_4: track 78.9 -> 0.00 mm
- net Net-(D6-Pad2): track 77.4 -> 0.00 mm
- net /DIGITAL_11: track 76.1 -> 0.00 mm
- net /DIGITAL_5: track 74.1 -> 0.00 mm
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Other:
- board text removed: "This is the underside of the PCB, which will not be seen. Solder in this order: resistors, diodes, IC socket, MIDI switch, 15-pin headers, capacitors, audio socket, power switch, buttons, LEDs, potentiometers, MIDI sockets, battery leads"

Commit message: smt pcb slowly happening
Parts:
- added U3: drumkid_logo, drumkidcustom:drumkid_logo, F.Cu at (100.5, 60.0)
- C1, C3: footprint Capacitor_SMD:CP_Elec_6.3x7.7 -> Capacitor_THT:CP_Radial_D6.3mm_P2.50mm
- C2, C5, D7, D8, R1, R10, R11, R12, R13, R14, R2, R3, R4, R5, R6, R7, R8, R9, U1: moved to B.Cu
- SW1, SW2, SW3, SW4, SW5, SW6: footprint drumkidcustom:SW_PUSH-12mm_Wuerth-430476085716 -> drumkidcustom:SW_Push_1P1T_NO_CK_PTS125Sx43PSMTR
- moved R12 53.7 mm to (81.0, 105.0), turned to 270 degrees
- moved R13 53.3 mm to (84.0, 105.0)
- moved R6 46.9 mm to (90.0, 105.0), turned to 90 degrees
- moved R5 46.9 mm to (93.0, 105.0), turned to 90 degrees
- moved R4 46.9 mm to (96.0, 105.0), turned to 90 degrees
- moved R3 46.9 mm to (99.0, 105.0), turned to 90 degrees
- moved R2 46.9 mm to (102.1, 105.0), turned to 90 degrees
- moved R1 46.9 mm to (105.0, 105.0), turned to 90 degrees
- moved C5 36.2 mm to (87.0, 112.0), turned to 180 degrees
- moved R7 32.3 mm to (122.0, 121.9), turned to 90 degrees
- moved R14 25.3 mm to (87.0, 105.0), turned to 90 degrees
- moved R8 19.1 mm to (106.0, 117.1)
- moved R9 16.3 mm to (106.0, 113.0)
- moved R11 10.8 mm to (89.0, 148.0), turned to 270 degrees
- moved D7 9.61 mm to (122.0, 116.3)
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Other:
- board text added: "DrumKid v11 by Matt Bradshaw mattbradshawdesign.com github.com/mattybrad/drumkid"
- board text removed: "DrumKid v10 by Matt Bradshaw mattbradshawdesign.com github.com/mattybrad/drumkid"
