File: pcb/v11/drumkid.kicad_pcb (KiCad board)
At the start: 2 copper layers, 90 x 140 mm, 69 parts, among them J1 DIN-5_180degree, J10 Conn_01x15, J11 Conn_01x15, J12 Conn_01x05, J13 AudioJack3_Ground_Switch, J14 Conn_01x05, J15 AudioJack3_Ground_Switch, J2 DIN-5_180degree, J3 Conn_01x15, J4 Conn_01x15, J5 Conn_01x10, J6 Conn_01x10, J7 Conn_01x10, J8 Conn_01x10, J9 AudioJack3_Ground_Switch, SW1 SW_Push, SW2 SW_Push, SW3 SW_Push, SW4 SW_Push, SW5 SW_Push, SW6 SW_Push, SW7 SW_SPDT, SW8 SW_SPDT, U1 6N138, U2 drumkid_logo, U3 drumkid_logo

Commit message: test led
Parts:
- added D9: LED, LED_SMD:LED_0805_2012Metric, F.Cu at (152.4, 158.8)
- added R15: 680*, Resistor_THT:R_Axial_DIN0207_L6.3mm_D2.5mm_P7.62mm_Horizontal, F.Cu at (151.7, 155.2)

Commit message: routing is hard
Parts:
- D9: moved to B.Cu
- moved D9 33.9 mm to (124.5, 139.5)
- moved R15 33.3 mm to (124.5, 136.0), turned to 90 degrees
- turned R1 to 270 degrees
- turned R2 to 270 degrees
- turned R3 to 270 degrees
- turned R4 to 270 degrees
- turned R5 to 270 degrees
- turned R6 to 270 degrees
Routing:
- net Net-(D8-Pad2): track 0.00 -> 192.0 mm
- net /ANALOG_0: track 0.00 -> 125.3 mm
- net VCC: track 0.00 -> 122.6 mm
- net /ANALOG_1: track 0.00 -> 118.7 mm
- net Net-(J9-PadT): track 0.00 -> 83.8 mm
- net /ANALOG_3: track 0.00 -> 82.7 mm
- net /DIGITAL_4: track 0.00 -> 81.6 mm, vias 0 -> 1
- net /ANALOG_2: track 0.00 -> 80.7 mm
- net Net-(C5-Pad1): track 0.00 -> 80.3 mm
- net Net-(BT1-Pad1): track 0.00 -> 71.1 mm
- net Net-(J9-PadR): track 0.00 -> 70.1 mm
- net /DIGITAL_5: track 0.00 -> 68.8 mm
- net Net-(D1-Pad2): track 0.00 -> 67.1 mm
- net Net-(D2-Pad2): track 0.00 -> 62.6 mm
- net Net-(D6-Pad2): track 0.00 -> 61.7 mm, vias 0 -> 2
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Other:
- board text removed: "1N4148"
- board text removed: "1N5817"

Commit message: better routing
Parts:
- moved R6 45.2 mm to (61.0, 139.7), turned to 0 degrees
- moved R4 28.7 mm to (68.6, 113.5)
- moved R5 28.3 mm to (66.0, 113.5)
- moved R14 15.8 mm to (73.7, 113.5), turned to 270 degrees
- moved R1 13.9 mm to (94.0, 113.5)
- moved R2 13.7 mm to (91.4, 113.5)
- moved R3 13.2 mm to (88.9, 113.5)
- moved R12 8.55 mm to (79.8, 113.5)
- moved R13 8.54 mm to (82.8, 113.5)
- moved C2 6.31 mm to (76.2, 112.5), turned to 0 degrees
- moved C3 5.81 mm to (97.3, 114.0)
- moved C5 1.41 mm to (86.4, 113.3), turned to 270 degrees
Routing:
- net VCC: track 122.6 -> 268.3 mm, vias 0 -> 2
- net Net-(C2-Pad1): track 11.2 -> 109.4 mm, vias 0 -> 2
- net Net-(D7-Pad2): track 4.41 -> 75.6 mm, vias 0 -> 2
- net Net-(J1-Pad4): track 0.00 -> 66.2 mm
- net GND: track 10.2 -> 73.0 mm, vias 0 -> 2
- net /DIGITAL_13: track 51.5 -> 9.22 mm, vias 2 -> 0
- net Net-(D2-Pad2): track 62.6 -> 103.6 mm, vias 0 -> 1
- net Net-(D6-Pad2): track 61.7 -> 101.1 mm, vias 2 -> 0
- net Net-(D1-Pad2): track 67.1 -> 96.0 mm
- net Net-(BT1-Pad1): track 71.1 -> 96.0 mm
- net /ANALOG_1: track 118.7 -> 143.1 mm
- net /DIGITAL_7: track 47.9 -> 71.4 mm
- net /ANALOG_2: track 80.7 -> 101.0 mm
- net Net-(D4-Pad2): track 55.9 -> 74.9 mm, vias 1 -> 3
- net /DIGITAL_9: track 25.9 -> 9.98 mm, vias 1 -> 0
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