File: pcb/v11/drumkid.sch (KiCad schematic (older format))
At the start: 69 parts, among them J1 DIN-5_180degree, J10 Conn_01x15, J11 Conn_01x15, J12 Conn_01x05, J13 AudioJack3_Ground_Switch, J14 Conn_01x05, J15 AudioJack3_Ground_Switch, J2 DIN-5_180degree, J3 Conn_01x15, J4 Conn_01x15, J5 Conn_01x10, J6 Conn_01x10, J7 Conn_01x10, J8 Conn_01x10, J9 AudioJack3_Ground_Switch, SW1 SW_Push, SW2 SW_Push, SW3 SW_Push, SW4 SW_Push, SW5 SW_Push, SW6 SW_Push, SW7 SW_SPDT, SW8 SW_SPDT, U1 6N138, U2 drumkid_logo, U3 drumkid_logo

Commit message: little manual update and new PCB in progress
Parts:
- C1, C3: footprint drumkidcustom:CP_Radial_D6.3mm_P2.50mm -> Capacitor_SMD:CP_Elec_6.3x7.7
- C2: footprint Capacitor_THT:C_Disc_D3.0mm_W1.6mm_P2.50mm -> Capacitor_SMD:C_0402_1005Metric
- C5: footprint drumkidcustom:CP_Radial_D6.3mm_P2.50mm -> Capacitor_SMD:C_0603_1608Metric
- D7: footprint Diode_THT:D_DO-35_SOD27_P7.62mm_Horizontal -> Diode_SMD:D_SOD-123
- D8: footprint Diode_THT:D_DO-41_SOD81_P10.16mm_Horizontal -> Diode_SMD:D_SOD-123
- R1, R10, R11, R12, R13, R14, R2, R3, R4, R5, R6, R7, R8, R9: footprint drumkidcustom:R_Axial_DIN0207_L6.3mm_D2.5mm_P10.16mm_Horizontal -> Resistor_SMD:R_0805_2012Metric
- U1: footprint Package_DIP:DIP-8_W7.62mm_Socket -> Package_DIP:PowerIntegrations_SMD-8
Changed lines of the file:
@@
 Title "DrumKid"
 Date ""
-Rev "v10"
+Rev "v11"
 Comp "by Matt Bradshaw"
 Comment1 ""
@@
 F 0 "D8" V 2246 1521 50  0000 R CNN
 F 1 "1N5817" V 2155 1521 50  0000 R CNN
-F 2 "Diode_THT:D_DO-41_SOD81_P10.16mm_Horizontal" H 2200 1425 50  0001 C CNN
+F 2 "Diode_SMD:D_SOD-123" H 2200 1425 50  0001 C CNN
 F 3 "http://www.vishay.com/docs/88525/1n5817.pdf" H 2200 1600 50  0001 C CNN
 	1    2200 1600
@@
 F 0 "R10" V 5743 5700 50  0000 C CNN
 F 1 "220" V 5834 5700 50  0000 C CNN
-F 2 "drumkidcustom:R_Axial_DIN0207_L6.3mm_D2.5mm_P10.16mm_Horizontal" V 5880 5700 50  0001 C CNN
+F 2 "Resistor_SMD:R_0805_2012Metric" V 5880 5700 50  0001 C CNN
 F 3 "~" H 5950 5700 50  0001 C CNN
 	1    5950 5700
@@
 F 0 "R11" V 6643 5700 50  0000 C CNN
 F 1 "220" V 6734 5700 50  0000 C CNN
-F 2 "drumkidcustom:R_Axial_DIN0207_L6.3mm_D2.5mm_P10.16mm_Horizontal" V 6780 5700 50  0001 C CNN
+F 2 "Resistor_SMD:R_0805_2012Metric" V 6780 5700 50  0001 C CNN
 F 3 "~" H 6850 5700 50  0001 C CNN
 	1    6850 5700
@@
 F 0 "R7" V 1143 5700 50  0000 C CNN
 F 1 "220" V 1234 5700 50  0000 C CNN
-F 2 "drumkidcustom:R_Axial_DIN0207_L6.3mm_D2.5mm_P10.16mm_Horizontal" V 1280 5700 50  0001 C CNN
+F 2 "Resistor_SMD:R_0805_2012Metric" V 1280 5700 50  0001 C CNN
 F 3 "~" H 1350 5700 50  0001 C CNN
 	1    1350 5700
@@
 F 0 "D7" V 1454 5929 50  0000 L CNN
 F 1 "1N4148" V 1545 5929 50  0000 L CNN
-F 2 "Diode_THT:D_DO-35_SOD27_P7.62mm_Horizontal" H 1500 5675 50  0001 C CNN
+F 2 "Diode_SMD:D_SOD-123" H 1500 5675 50  0001 C CNN
 F 3 "http://www.nxp.com/documents/data_sheet/1N4148_1N4448.pdf" H 1500 5850 50  0001 C CNN
 	1    1500 5850
@@
 F 0 "U1" H 2350 6267 50  0000 C CNN
 F 1 "6N138" H 2350 6176 50  0000 C CNN
-F 2 "Package_DIP:DIP-8_W7.62mm_Socket" H 2640 5500 50  0001 C CNN
+F 2 "Package_DIP:PowerIntegrations_SMD-8" H 2640 5500 50  0001 C CNN
 F 3 "http://www.onsemi.com/pub/Collateral/HCPL2731-D.pdf" H 2640 5500 50  0001 C CNN
 	1    2350 5800
@@
 F 0 "R9" V 4193 5900 50  0000 C CNN
 F 1 "470" V 4284 5900 50  0000 C CNN
-F 2 "drumkidcustom:R_Axial_DIN0207_L6.3mm_D2.5mm_P10.16mm_Horizontal" V 4330 5900 50  0001 C CNN
+F 2 "Resistor_SMD:R_0805_2012Metric" V 4330 5900 50  0001 C CNN
 F 3 "~" H 4400 5900 50  0001 C CNN
 	1    4400 5900
@@
 F 0 "R8" V 2593 5700 50  0000 C CNN
 F 1 "10k" V 2684 5700 50  0000 C CNN
-F 2 "drumkidcustom:R_Axial_DIN0207_L6.3mm_D2.5mm_P10.16mm_Horizontal" V 2730 5700 50  0001 C CNN
+F 2 "Resistor_SMD:R_0805_2012Metric" V 2730 5700 50  0001 C CNN
 F 3 "~" H 2800 5700 50  0001 C CNN
 	1    2800 5700
@@
 F 0 "R1" V 5243 1650 50  0000 C CNN
 F 1 "680*" V 5334 1650 50  0000 C CNN
-F 2 "drumkidcustom:R_Axial_DIN0207_L6.3mm_D2.5mm_P10.16mm_Horizontal" V 5380 1650 50  0001 C CNN
+F 2 "Resistor_SMD:R_0805_2012Metric" V 5380 1650 50  0001 C CNN
 F 3 "~" H 5450 1650 50  0001 C CNN
 	1    5450 1650
@@
 F 0 "C1" H 3068 1396 50  0000 L CNN
 F 1 "470uF" H 3068 1305 50  0000 L CNN
-F 2 "drumkidcustom:CP_Radial_D6.3mm_P2.50mm" H 2988 1200 50  0001 C CNN
+F 2 "Capacitor_SMD:CP_Elec_6.3x7.7" H 2988 1200 50  0001 C CNN
 F 3 "~" H 2950 1350 50  0001 C CNN
 	1    2950 1350
@@
 F 0 "C3" H 4918 5596 50  0000 L CNN
 F 1 "470uF" H 4918 5505 50  0000 L CNN
-F 2 "drumkidcustom:CP_Radial_D6.3mm_P2.50mm" H 4838 5400 50  0001 C CNN
+F 2 "Capacitor_SMD:CP_Elec_6.3x7.7" H 4838 5400 50  0001 C CNN
 F 3 "~" H 4800 5550 50  0001 C CNN
 	1    4800 5550
@@
 F 0 "C5" V 9255 5300 50  0000 C CNN
 F 1 "22uF" V 9164 5300 50  0000 C CNN
-F 2 "drumkidcustom:CP_Radial_D6.3mm_P2.50mm" H 9038 5150 50  0001 C CNN
+F 2 "Capacitor_SMD:C_0603_1608Metric" H 9038 5150 50  0001 C CNN
 F 3 "~" H 9000 5300 50  0001 C CNN
 	1    9000 5300
@@
 F 0 "R13" V 9850 5500 50  0000 C CNN
 F 1 "220" V 9950 5500 50  0000 C CNN
-F 2 "drumkidcustom:R_Axial_DIN0207_L6.3mm_D2.5mm_P10.16mm_Horizontal" V 9680 5500 50  0001 C CNN
+F 2 "Resistor_SMD:R_0805_2012Metric" V 9680 5500 50  0001 C CNN
 F 3 "~" H 9750 5500 50  0001 C CNN
 	1    9750 5500
@@
 F 0 "R12" V 9543 5300 50  0000 C CNN
 F 1 "220" V 9634 5300 50  0000 C CNN
-F 2 "drumkidcustom:R_Axial_DIN0207_L6.3mm_D2.5mm_P10.16mm_Horizontal" V 9680 5300 50  0001 C CNN
+F 2 "Resistor_SMD:R_0805_2012Metric" V 9680 5300 50  0001 C CNN
 F 3 "~" H 9750 5300 50  0001 C CNN
 	1    9750 5300
@@
 F 0 "R14" V 7843 5600 50  0000 C CNN
 F 1 "270" V 7934 5600 50  0000 C CNN
-F 2 "drumkidcustom:R_Axial_DIN0207_L6.3mm_D2.5mm_P10.16mm_Horizontal" V 7980 5600 50  0001 C CNN
+F 2 "Resistor_SMD:R_0805_2012Metric" V 7980 5600 50  0001 C CNN
 F 3 "~" H 8050 5600 50  0001 C CNN
 	1    8050 5600
@@
 F 0 "C2" H 8415 5896 50  0000 L CNN
 F 1 "100nF" H 8415 5805 50  0000 L CNN
-F 2 "Capacitor_THT:C_Disc_D3.0mm_W1.6mm_P2.50mm" H 8338 5700 50  0001 C CNN
+F 2 "Capacitor_SMD:C_0402_1005Metric" H 8338 5700 50  0001 C CNN
 F 3 "~" H 8300 5850 50  0001 C CNN
 	1    8300 5850
@@
 F 0 "R2" V 5243 2050 50  0000 C CNN
 F 1 "680*" V 5334 2050 50  0000 C CNN
-F 2 "drumkidcustom:R_Axial_DIN0207_L6.3mm_D2.5mm_P10.16mm_Horizontal" V 5380 2050 50  0001 C CNN
+F 2 "Resistor_SMD:R_0805_2012Metric" V 5380 2050 50  0001 C CNN
 F 3 "~" H 5450 2050 50  0001 C CNN
 	1    5450 2050
@@
 F 0 "R3" V 5243 2450 50  0000 C CNN
 F 1 "680*" V 5334 2450 50  0000 C CNN
-F 2 "drumkidcustom:R_Axial_DIN0207_L6.3mm_D2.5mm_P10.16mm_Horizontal" V 5380 2450 50  0001 C CNN
+F 2 "Resistor_SMD:R_0805_2012Metric" V 5380 2450 50  0001 C CNN
 F 3 "~" H 5450 2450 50  0001 C CNN
 	1    5450 2450
@@
 F 0 "R5" V 5243 3250 50  0000 C CNN
 F 1 "680*" V 5334 3250 50  0000 C CNN
-F 2 "drumkidcustom:R_Axial_DIN0207_L6.3mm_D2.5mm_P10.16mm_Horizontal" V 5380 3250 50  0001 C CNN
+F 2 "Resistor_SMD:R_0805_2012Metric" V 5380 3250 50  0001 C CNN
 F 3 "~" H 5450 3250 50  0001 C CNN
 	1    5450 3250
@@
 F 0 "R6" V 5243 3650 50  0000 C CNN
 F 1 "680*" V 5334 3650 50  0000 C CNN
-F 2 "drumkidcustom:R_Axial_DIN0207_L6.3mm_D2.5mm_P10.16mm_Horizontal" V 5380 3650 50  0001 C CNN
+F 2 "Resistor_SMD:R_0805_2012Metric" V 5380 3650 50  0001 C CNN
 F 3 "~" H 5450 3650 50  0001 C CNN
 	1    5450 3650
@@
 F 0 "R4" V 5243 2850 50  0000 C CNN
 F 1 "680*" V 5334 2850 50  0000 C CNN
-F 2 "drumkidcustom:R_Axial_DIN0207_L6.3mm_D2.5mm_P10.16mm_Horizontal" V 5380 2850 50  0001 C CNN
+F 2 "Resistor_SMD:R_0805_2012Metric" V 5380 2850 50  0001 C CNN
 F 3 "~" H 5450 2850 50  0001 C CNN
 	1    5450 2850

Commit message: smt pcb slowly happening
Parts:
- C1, C3: footprint Capacitor_SMD:CP_Elec_6.3x7.7 -> Capacitor_THT:CP_Radial_D6.3mm_P2.50mm
- SW1, SW2, SW3, SW4, SW5, SW6: footprint drumkidcustom:SW_PUSH-12mm_Wuerth-430476085716 -> drumkidcustom:SW_Push_1P1T_NO_CK_PTS125Sx43PSMTR
Changed lines of the file:
@@
 F 0 "SW1" H 4300 1935 50  0000 C CNN
 F 1 "SW_Push" H 4300 1844 50  0000 C CNN
-F 2 "drumkidcustom:SW_PUSH-12mm_Wuerth-430476085716" H 4300 1850 50  0001 C CNN
+F 2 "drumkidcustom:SW_Push_1P1T_NO_CK_PTS125Sx43PSMTR" H 4300 1850 50  0001 C CNN
 F 3 "" H 4300 1850 50  0001 C CNN
 	1    4300 1650
@@
 F 0 "SW2" H 4300 2335 50  0000 C CNN
 F 1 "SW_Push" H 4300 2244 50  0000 C CNN
-F 2 "drumkidcustom:SW_PUSH-12mm_Wuerth-430476085716" H 4300 2250 50  0001 C CNN
+F 2 "drumkidcustom:SW_Push_1P1T_NO_CK_PTS125Sx43PSMTR" H 4300 2250 50  0001 C CNN
 F 3 "" H 4300 2250 50  0001 C CNN
 	1    4300 2050
@@
 F 0 "SW3" H 4300 2735 50  0000 C CNN
 F 1 "SW_Push" H 4300 2644 50  0000 C CNN
-F 2 "drumkidcustom:SW_PUSH-12mm_Wuerth-430476085716" H 4300 2650 50  0001 C CNN
+F 2 "drumkidcustom:SW_Push_1P1T_NO_CK_PTS125Sx43PSMTR" H 4300 2650 50  0001 C CNN
 F 3 "" H 4300 2650 50  0001 C CNN
 	1    4300 2450
@@
 F 0 "SW4" H 4300 3135 50  0000 C CNN
 F 1 "SW_Push" H 4300 3044 50  0000 C CNN
-F 2 "drumkidcustom:SW_PUSH-12mm_Wuerth-430476085716" H 4300 3050 50  0001 C CNN
+F 2 "drumkidcustom:SW_Push_1P1T_NO_CK_PTS125Sx43PSMTR" H 4300 3050 50  0001 C CNN
 F 3 "" H 4300 3050 50  0001 C CNN
 	1    4300 2850
@@
 F 0 "SW5" H 4300 3535 50  0000 C CNN
 F 1 "SW_Push" H 4300 3444 50  0000 C CNN
-F 2 "drumkidcustom:SW_PUSH-12mm_Wuerth-430476085716" H 4300 3450 50  0001 C CNN
+F 2 "drumkidcustom:SW_Push_1P1T_NO_CK_PTS125Sx43PSMTR" H 4300 3450 50  0001 C CNN
 F 3 "" H 4300 3450 50  0001 C CNN
 	1    4300 3250
@@
 F 0 "SW6" H 4300 3935 50  0000 C CNN
 F 1 "SW_Push" H 4300 3844 50  0000 C CNN
-F 2 "drumkidcustom:SW_PUSH-12mm_Wuerth-430476085716" H 4300 3850 50  0001 C CNN
+F 2 "drumkidcustom:SW_Push_1P1T_NO_CK_PTS125Sx43PSMTR" H 4300 3850 50  0001 C CNN
 F 3 "" H 4300 3850 50  0001 C CNN
 	1    4300 3650
@@
 F 0 "C1" H 3068 1396 50  0000 L CNN
 F 1 "470uF" H 3068 1305 50  0000 L CNN
-F 2 "Capacitor_SMD:CP_Elec_6.3x7.7" H 2988 1200 50  0001 C CNN
+F 2 "Capacitor_THT:CP_Radial_D6.3mm_P2.50mm" H 2988 1200 50  0001 C CNN
 F 3 "~" H 2950 1350 50  0001 C CNN
 	1    2950 1350
@@
 F 0 "C3" H 4918 5596 50  0000 L CNN
 F 1 "470uF" H 4918 5505 50  0000 L CNN
-F 2 "Capacitor_SMD:CP_Elec_6.3x7.7" H 4838 5400 50  0001 C CNN
+F 2 "Capacitor_THT:CP_Radial_D6.3mm_P2.50mm" H 4838 5400 50  0001 C CNN
 F 3 "~" H 4800 5550 50  0001 C CNN
 	1    4800 5550

Commit message: test led
Parts:
- added D9: LED, LED_SMD:LED_0805_2012Metric, symbol Device:LED
- added R15: 680*, Resistor_THT:R_Axial_DIN0207_L6.3mm_D2.5mm_P7.62mm_Horizontal, symbol Device:R
Connections:
- net GND: now also D9.1 (K)
- net VCC: now also R15.2
- new net: D9.2 (A), R15.1
Other:
- moved on the sheet: D1, D2, D3, D4, D5, D6, R1, R2, R3, R4, R5, R6

Commit message: v11 done and ordered
Parts:
- R1, R15, R2, R3, R4, R5, R6: value 680* -> 680
Changed lines of the file:
@@
 P 5550 2150
 F 0 "R1" V 5343 2150 50  0000 C CNN
-F 1 "680*" V 5434 2150 50  0000 C CNN
+F 1 "680" V 5434 2150 50  0000 C CNN
 F 2 "Resistor_SMD:R_0805_2012Metric" V 5480 2150 50  0001 C CNN
 F 3 "~" H 5550 2150 50  0001 C CNN
@@
 P 5550 2550
 F 0 "R2" V 5343 2550 50  0000 C CNN
-F 1 "680*" V 5434 2550 50  0000 C CNN
+F 1 "680" V 5434 2550 50  0000 C CNN
 F 2 "Resistor_SMD:R_0805_2012Metric" V 5480 2550 50  0001 C CNN
 F 3 "~" H 5550 2550 50  0001 C CNN
@@
 P 5550 2950
 F 0 "R3" V 5343 2950 50  0000 C CNN
-F 1 "680*" V 5434 2950 50  0000 C CNN
+F 1 "680" V 5434 2950 50  0000 C CNN
 F 2 "Resistor_SMD:R_0805_2012Metric" V 5480 2950 50  0001 C CNN
 F 3 "~" H 5550 2950 50  0001 C CNN
@@
 P 5550 3750
 F 0 "R5" V 5343 3750 50  0000 C CNN
-F 1 "680*" V 5434 3750 50  0000 C CNN
+F 1 "680" V 5434 3750 50  0000 C CNN
 F 2 "Resistor_SMD:R_0805_2012Metric" V 5480 3750 50  0001 C CNN
 F 3 "~" H 5550 3750 50  0001 C CNN
@@
 P 5550 4150
 F 0 "R6" V 5343 4150 50  0000 C CNN
-F 1 "680*" V 5434 4150 50  0000 C CNN
+F 1 "680" V 5434 4150 50  0000 C CNN
 F 2 "Resistor_SMD:R_0805_2012Metric" V 5480 4150 50  0001 C CNN
 F 3 "~" H 5550 4150 50  0001 C CNN
@@
 P 5550 3350
 F 0 "R4" V 5343 3350 50  0000 C CNN
-F 1 "680*" V 5434 3350 50  0000 C CNN
+F 1 "680" V 5434 3350 50  0000 C CNN
 F 2 "Resistor_SMD:R_0805_2012Metric" V 5480 3350 50  0001 C CNN
 F 3 "~" H 5550 3350 50  0001 C CNN
@@
 P 5550 1750
 F 0 "R15" V 5343 1750 50  0000 C CNN
-F 1 "680*" V 5434 1750 50  0000 C CNN
+F 1 "680" V 5434 1750 50  0000 C CNN
 F 2 "Resistor_THT:R_Axial_DIN0207_L6.3mm_D2.5mm_P7.62mm_Horizontal" V 5480 1750 50  0001 C CNN
 F 3 "~" H 5550 1750 50  0001 C CNN
