File: pcb/v13/drumkid.kicad_pcb (KiCad board)
At the start: 2 copper layers, 90 x 140 mm, 68 parts, among them J1 DIN-5_180degree, J10 Conn_01x15, J11 Conn_01x15, J12 Conn_01x05, J13 AudioJack3_Ground_Switch, J14 Conn_01x05, J15 AudioJack3_Ground_Switch, J2 DIN-5_180degree, J3 Conn_01x15, J4 Conn_01x15, J5 Conn_01x10, J6 Conn_01x10, J7 Conn_01x10, J8 Conn_01x10, J9 AudioJack3_Ground_Switch, SW1 SW_Push, SW2 SW_Push, SW3 SW_Push, SW4 SW_Push, SW5 SW_Push, SW6 SW_Push, SW7 SW_SPDT, SW8 SW_SPDT, U1 6N138, U2 drumkid_logo

Commit message: oh wow i haven't updated for ages
Routing:
- net Net-(J9-PadT): track 92.8 -> 95.7 mm
- net Net-(J9-PadR): track 82.0 -> 84.4 mm
Changed lines of the file:
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@@
     (thickness 1.6)
     (drawings 119)
-    (tracks 488)
+    (tracks 499)
     (zones 0)
     (modules 68)
@@
   (segment (start 87.376 112.62015) (end 87.376 114.273994) (width 0.25) (layer B.Cu) (net 38))
   (segment (start 95 104.99615) (end 87.376 112.62015) (width 0.25) (layer B.Cu) (net 38))
-  (segment (start 95 40.41) (end 95 104.99615) (width 0.25) (layer B.Cu) (net 38))
+  (segment (start 95 48.353002) (end 95 42.41) (width 0.25) (layer B.Cu) (net 38))
+  (segment (start 92.13099 51.222012) (end 95 48.353002) (width 0.25) (layer B.Cu) (net 38))
+  (segment (start 92.13099 59.824626) (end 92.13099 51.222012) (width 0.25) (layer B.Cu) (net 38))
+  (segment (start 95 62.693636) (end 92.13099 59.824626) (width 0.25) (layer B.Cu) (net 38))
+  (segment (start 95 42.41) (end 95 40.41) (width 0.25) (layer B.Cu) (net 38))
+  (segment (start 95 104.99615) (end 95 62.693636) (width 0.25) (layer B.Cu) (net 38))
   (segment (start 94.829999 133.770001) (end 93.98 134.62) (width 0.625) (layer B.Cu) (net 39))
   (segment (start 105.542501 121.246799) (end 105.542501 123.057499) (width 0.625) (layer B.Cu) (net 39))
@@
   (segment (start 118.065001 67.991999) (end 118.065001 79.912399) (width 0.25) (layer F.Cu) (net 57))
   (segment (start 93.79999 98.47801) (end 80.241527 112.036473) (width 0.25) (layer B.Cu) (net 58))
-  (segment (start 93.79999 39.03794) (end 93.79999 98.47801) (width 0.25) (layer B.Cu) (net 58))
   (segment (start 104.92499 38.33499) (end 94.50294 38.33499) (width 0.25) (layer B.Cu) (net 58))
   (segment (start 94.50294 38.33499) (end 93.79999 39.03794) (width 0.25) (layer B.Cu) (net 58))
@@
   (segment (start 80.241527 112.036473) (end 79.756 112.522) (width 0.25) (layer B.Cu) (net 58))
   (segment (start 105 40.41) (end 105 38.41) (width 0.25) (layer B.Cu) (net 58))
+  (segment (start 90.314999 77.757599) (end 93.79999 81.24259) (width 0.25) (layer B.Cu) (net 58))
+  (segment (start 90.314999 47.585001) (end 90.314999 77.757599) (width 0.25) (layer B.Cu) (net 58))
+  (segment (start 93.79999 81.24259) (end 93.79999 98.47801) (width 0.25) (layer B.Cu) (net 58))
+  (segment (start 93.79999 44.10001) (end 90.314999 47.585001) (width 0.25) (layer B.Cu) (net 58))
+  (segment (start 93.79999 39.03794) (end 93.79999 44.10001) (width 0.25) (layer B.Cu) (net 58))
   (segment (start 73.7385 112.522) (end 73.66 112.6005) (width 0.25) (layer B.Cu) (net 59))
   (segment (start 75.738 112.522) (end 73.7385 112.522) (width 0.25) (layer B.Cu) (net 59))
   (segment (start 75.384502 112.6005) (end 74.36 112.6005) (width 0.25) (layer B.Cu) (net 59))
-  (segment (start 94.316539 37.884981) (end 92.765001 39.436519) (width 0.25) (layer B.Cu) (net 59))
-  (segment (start 108.884981 37.884981) (end 94.316539 37.884981) (width 0.25) (layer B.Cu) (net 59))
   (segment (start 74.36 112.6005) (end 73.66 112.6005) (width 0.25) (layer B.Cu) (net 59))
-  (segment (start 115 44) (end 108.884981 37.884981) (width 0.25) (layer B.Cu) (net 59))
   (via (at 79.793143 105.066993) (size 0.8) (drill 0.4) (layers F.Cu B.Cu) (net 59))
   (segment (start 75.738 112.522) (end 75.738 112.202) (width 0.25) (layer B.Cu) (net 59))
@@
   (via (at 87.884 70.358) (size 0.8) (drill 0.4) (layers F.Cu B.Cu) (net 59))
   (segment (start 79.793143 105.066993) (end 87.884 96.976136) (width 0.25) (layer F.Cu) (net 59))
-  (segment (start 92.765001 57.911001) (end 92.765001 39.436519) (width 0.25) (layer B.Cu) (net 59))
-  (segment (start 87.884 62.792002) (end 92.765001 57.911001) (width 0.25) (layer B.Cu) (net 59))
-  (segment (start 87.884 70.358) (end 87.884 62.792002) (width 0.25) (layer B.Cu) (net 59))
   (segment (start 88.283999 94.333401) (end 88.283999 70.757999) (width 0.25) (layer F.Cu) (net 59))
   (segment (start 87.884 96.976136) (end 87.884 94.7334) (width 0.25) (layer F.Cu) (net 59))
   (segment (start 88.283999 70.757999) (end 87.884 70.358) (width 0.25) (layer F.Cu) (net 59))
   (segment (start 87.884 94.7334) (end 88.283999 94.333401) (width 0.25) (layer F.Cu) (net 59))
+  (segment (start 87.965001 60.478999) (end 87.965001 62.711001) (width 0.25) (layer B.Cu) (net 59))
+  (segment (start 115 44) (end 108.884981 37.884981) (width 0.25) (layer B.Cu) (net 59))
+  (segment (start 87.884 62.792002) (end 87.884 70.358) (width 0.25) (layer B.Cu) (net 59))
+  (segment (start 87.965001 62.711001) (end 87.884 62.792002) (width 0.25) (layer B.Cu) (net 59))
+  (segment (start 94.316539 37.884981) (end 87.774999 44.426521) (width 0.25) (layer B.Cu) (net 59))
+  (segment (start 87.774999 60.288997) (end 87.965001 60.478999) (width 0.25) (layer B.Cu) (net 59))
+  (segment (start 108.884981 37.884981) (end 94.316539 37.884981) (width 0.25) (layer B.Cu) (net 59))
+  (segment (start 87.774999 44.426521) (end 87.774999 60.288997) (width 0.25) (layer B.Cu) (net 59))
   (segment (start 132.08 146.117919) (end 132.08 144.78) (width 0.25) (layer B.Cu) (net 60))
   (segment (start 132.08 147.32) (end 132.08 146.117919) (width 0.25) (layer B.Cu) (net 60))
@@
       )
     )
+  )
+  (zone (net 0) (net_name "") (layer B.Cu) (hatch edge 0.508)
+    (connect_pads (clearance 0.508))
+    (min_thickness 0.254)
+    (keepout (tracks not_allowed) (vias not_allowed) (copperpour not_allowed))
+    (fill (arc_segments 32) (thermal_gap 0.508) (thermal_bridge_width 0.508))
+    (polygon
+      (pts
+        (xy 95.25 59.69) (xy 92.456 59.69) (xy 92.456 56.896) (xy 95.25 56.896)
+      )
+    )
