File: pcb/v14/drumkid.kicad_pcb (KiCad board)
At the start: 2 copper layers, 90 x 140 mm, 68 parts, among them J1 DIN-5_180degree, J10 Conn_01x15, J11 Conn_01x15, J12 Conn_01x05, J13 AudioJack3_Ground_Switch, J14 Conn_01x05, J15 AudioJack3_Ground_Switch, J2 DIN-5_180degree, J3 Conn_01x15, J4 Conn_01x15, J5 Conn_01x10, J6 Conn_01x10, J7 Conn_01x10, J8 Conn_01x10, J9 AudioJack3_Ground_Switch, SW1 SW_Push, SW2 SW_Push, SW3 SW_Push, SW4 SW_Push, SW5 SW_Push, SW6 SW_Push, SW7 SW_SPDT, SW8 SW_SPDT, U1 6N138, U2 drumkid_logo

Commit message: things have happened. bad things?
Parts:
- added U3: drumkid_logo, drumkidcustom:drumkid_logo, F.Cu at (100.5, 60.0)
- U1: footprint Package_DIP:DIP-8_W7.62mm_Socket -> Package_DIP:PowerIntegrations_SMD-8; moved to B.Cu
- moved U1 6.39 mm to (114.0, 116.0), turned to 180 degrees
Routing:
- net GND: track 44.0 -> 73.0 mm, vias 0 -> 2
- net VCC: track 253.8 -> 268.3 mm
- net Net-(D7-Pad2): track 88.5 -> 75.6 mm, vias 1 -> 2
- net Net-(D7-Pad1): track 24.7 -> 14.1 mm
- net Net-(R8-Pad2): track 11.6 -> 4.28 mm
- net Net-(R9-Pad2): track 43.9 -> 37.5 mm
- net Net-(D9-Pad2): track 0.00 -> 3.89 mm
- net Net-(J9-PadT): track 95.7 -> 92.8 mm
- net Net-(J9-PadR): track 84.4 -> 82.0 mm
Other:
- net class Chunky removed
- net class Default removed
- board text added: "DrumKid v12 by Matt Bradshaw mattbradshawdesign.com github.com/mattybrad/drumkid"
- board text removed: "DrumKid v13 by Matt Bradshaw mattbradshawdesign.com github.com/mattybrad/drumkid"
- board text removed: "Soldering order: 1) 6N138 socket 2) MIDI switch 3) 15-pin headers 4) Capacitors 5) Audio socket 6) Power switch 7) Buttons 8) LEDs 9) Potentiometers 10) MIDI sockets 11) Battery leads"
