File: pcb/v14/drumkid.kicad_sch (KiCad schematic)
At the start: 70 parts, among them J1 DIN-5_180degree, J10 Conn_01x15, J11 Conn_01x15, J12 Conn_01x05, J13 AudioJack3_Ground_Switch, J14 Conn_01x05, J15 AudioJack3_Ground_Switch, J2 DIN-5_180degree, J3 Conn_01x15, J4 Conn_01x15, J5 Conn_01x10, J6 Conn_01x10, J7 Conn_01x10, J8 Conn_01x10, J9 AudioJack3_Ground_Switch, SW1 SW_Push, SW2 SW_Push, SW3 SW_Push, SW4 SW_Push, SW5 SW_Push, SW6 SW_Push, SW7 SW_SPDT, SW8 SW_SPDT, U1 6N138, U2 drumkid_logo, U3 drumkid_logo

Commit message: things have happened. bad things?
Parts:
- removed U?: Pico, RPi_Pico:RPi_Pico_SMD_TH, symbol MCU_RaspberryPi_and_Boards:Pico
- A1: value Arduino_Nano_v3.x -> (none); footprint Module:Arduino_Nano_WithMountingHoles -> (none)
- BT1: value Battery -> (none); footprint Connector_Wire:SolderWirePad_1x02_P5.08mm_Drill1.5mm -> (none)
- C1, C3: value 470uF -> (none); footprint Capacitor_THT:CP_Radial_D6.3mm_P2.50mm -> (none); symbol Device:CP -> drumkid-rescue:CP-Device
- C2: value 100nF -> (none); footprint Capacitor_SMD:C_0402_1005Metric -> (none)
- C5: value 22uF -> (none); footprint Capacitor_SMD:C_0603_1608Metric -> (none); symbol Device:CP -> drumkid-rescue:CP-Device
- D1, D2, D3, D4, D5, D6: value LED -> (none); footprint drumkidcustom:LED_D5.0mm -> (none)
- D7: value 1N4148 -> (none); footprint Diode_SMD:D_SOD-123 -> (none)
- D8: value 1N5817 -> (none); footprint Diode_SMD:D_SOD-123 -> (none)
- H1, H10, H2, H3, H4, H5, H6, H7, H8, H9: value MountingHole -> (none); footprint drumkidcustom:MountingHole_3.2mm_M3 -> (none)
- J1, J2: value DIN-5_180degree -> (none); footprint drumkidcustom:MIDI_DIN5 -> (none)
- J10, J11: value Conn_01x15 -> (none); footprint Connector_PinHeader_2.54mm:PinHeader_1x15_P2.54mm_Vertical -> (none)
- J12, J14: value Conn_01x05 -> (none); footprint Connector_PinSocket_2.54mm:PinSocket_1x05_P2.54mm_Vertical -> (none)
- J13, J15, J9: value AudioJack3_Ground_Switch -> (none); footprint drumkidcustom:Tayda_3.5mm_stereo_TRS_jack_A-853 -> (none)
- J3, J4: value Conn_01x15 -> (none); footprint Connector_PinSocket_2.54mm:PinSocket_1x15_P2.54mm_Vertical -> (none)
- J5, J8: value Conn_01x10 -> (none); footprint Connector_PinSocket_2.54mm:PinSocket_1x10_P2.54mm_Vertical -> (none)
- J6, J7: value Conn_01x10 -> (none); footprint Connector_PinHeader_2.54mm:PinHeader_1x10_P2.54mm_Vertical -> (none)
- R1, R2, R3, R4, R5, R6: value 680 -> (none); footprint Resistor_SMD:R_0805_2012Metric -> (none)
- R10, R11, R12, R13, R7: value 220 -> (none); footprint Resistor_SMD:R_0805_2012Metric -> (none)
- R14: value 270 -> (none); footprint Resistor_SMD:R_0805_2012Metric -> (none)
- R8: value 10k -> (none); footprint Resistor_SMD:R_0805_2012Metric -> (none)
- R9: value 470 -> (none); footprint Resistor_SMD:R_0805_2012Metric -> (none)
- RV1, RV2, RV3, RV4: value R_POT -> (none); footprint drumkidcustom:Potentiometer_Alps_RK09K_Single_Vertical -> (none); symbol Device:R_POT -> drumkid-rescue:R_POT-Device
- RV5: value 10k -> (none); footprint drumkidcustom:Potentiometer_Alps_RK09K_Single_Vertical -> (none); symbol Device:R_POT -> drumkid-rescue:R_POT-Device
- SW1, SW2, SW3, SW4, SW5, SW6: value SW_Push -> (none); footprint drumkidcustom:SW_PUSH-12mm_Wuerth-430476085716 -> (none)
- SW7, SW8: value SW_SPDT -> (none); footprint drumkidcustom:EG1206 -> (none)
- U1: value 6N138 -> (none); footprint Package_DIP:DIP-8_W7.62mm_Socket -> (none)
- U2, U3: value drumkid_logo -> (none); footprint drumkidcustom:drumkid_logo -> (none)
