File: pcb/v12/drumkid.kicad_pcb (KiCad board)
At the start: 2 copper layers, 90 x 140 mm, 69 parts, among them J1 DIN-5_180degree, J10 Conn_01x15, J11 Conn_01x15, J12 Conn_01x05, J13 AudioJack3_Ground_Switch, J14 Conn_01x05, J15 AudioJack3_Ground_Switch, J2 DIN-5_180degree, J3 Conn_01x15, J4 Conn_01x15, J5 Conn_01x10, J6 Conn_01x10, J7 Conn_01x10, J8 Conn_01x10, J9 AudioJack3_Ground_Switch, SW1 SW_Push, SW2 SW_Push, SW3 SW_Push, SW4 SW_Push, SW5 SW_Push, SW6 SW_Push, SW7 SW_SPDT, SW8 SW_SPDT, U1 6N138, U2 drumkid_logo, U3 drumkid_logo

Commit message: about to update to kicad 7, fingers crossed
Other:
- net class Chunky removed
- net class Default removed
