File: pcb/v12/drumkid.kicad_pcb (KiCad board)
At the start: 2 copper layers, 90 x 140 mm, 69 parts, among them J1 DIN-5_180degree, J10 Conn_01x15, J11 Conn_01x15, J12 Conn_01x05, J13 AudioJack3_Ground_Switch, J14 Conn_01x05, J15 AudioJack3_Ground_Switch, J2 DIN-5_180degree, J3 Conn_01x15, J4 Conn_01x15, J5 Conn_01x10, J6 Conn_01x10, J7 Conn_01x10, J8 Conn_01x10, J9 AudioJack3_Ground_Switch, SW1 SW_Push, SW2 SW_Push, SW3 SW_Push, SW4 SW_Push, SW5 SW_Push, SW6 SW_Push, SW7 SW_SPDT, SW8 SW_SPDT, U1 6N138, U2 drumkid_logo, U3 drumkid_logo

Commit message: things
Connections:
- J1 pad 1: Net-(J1-Pad1) -> unconnected-(J1-Pad1)
- J1 pad 2: Net-(J1-Pad2) -> unconnected-(J1-Pad2)
- J1 pad 3: Net-(J1-Pad3) -> unconnected-(J1-Pad3)
- J2 pad 1: Net-(J2-Pad1) -> unconnected-(J2-Pad1)
- J2 pad 3: Net-(J2-Pad3) -> unconnected-(J2-Pad3)
- J9 pad RN: Net-(J9-PadRN) -> unconnected-(J9-PadRN)
- J9 pad TN: Net-(J9-PadTN) -> unconnected-(J9-PadTN)
- SW7 pad 3: Net-(SW7-Pad3) -> unconnected-(SW7-Pad3)
- SW8 pad 3: Net-(SW8-Pad3) -> unconnected-(SW8-Pad3)
- U1 pad 1: Net-(U1-Pad1) -> unconnected-(U1-Pad1)
- U1 pad 4: Net-(U1-Pad4) -> unconnected-(U1-Pad4)
Routing:
- net VCC: track 268.3 -> 245.6 mm
- net GND: track 73.0 -> 64.4 mm, vias 2 -> 0
- net Net-(D9-Pad2): track 3.89 -> 0.00 mm
- net Net-(J9-PadR): track 82.0 -> 84.3 mm
- net Net-(J9-PadT): track 92.8 -> 94.6 mm
- net /DIGITAL_10: track 50.7 -> 49.2 mm
- net Net-(BT1-Pad1): track 96.0 -> 97.1 mm
- net Net-(D8-Pad2): track 191.8 -> 192.9 mm
- net /DIGITAL_7: track 73.1 -> 72.1 mm
- net /ANALOG_2: track 101.3 -> 102.2 mm
- net /DIGITAL_5: track 67.0 -> 66.3 mm
Other:
- net class Chunky removed
- net class Default removed
- board text added: "DrumKid v15 by Matt Bradshaw bradshawinstruments.com github.com/mattybrad/drumkid"
- board text added: "bradshaw instruments"
- board text removed: "DrumKid v12 by Matt Bradshaw mattbradshawdesign.com github.com/mattybrad/drumkid"
- board text removed: "aleatoric drum machine"
